File: hardware/power/power_board.sch (EAGLE design)
At the start: 6 parts, among them J1 FASTON_MALE_RA_BLADE, J2 FASTON_MALE_RA_BLADE, J3 12v, J4 5v, U1 PDQ30-Q24-S5-D, U2 PDQ30-Q24-S12-D

Commit message: Power updates
Parts:
- added J5, J6, J7, J8: XT30PW-F, timlib:XT30PW-F
- added R1: 100, rcl:R-US_R0603
- added U$10, U$9: 2, timlib:PWR163
- added U$11: PSMN1R0-40YSH, timlib:PSMN1R0-40YSH
Connections:
- new net N$1: U$10.1, U$11.D
- net +24V: now also J5.V+, J6.V+, J7.V+, J8.V+
- net GND: now also J5.V-, J6.V-, J7.V-, J8.V-, U$11.S
Other:
- moved on the sheet: U1, U2

Commit message: Power board updates
Parts:
- added R2, R5: 2, timlib:PWR163
- added R4: 100, rcl:R-US_R0603
- added U$12: SMAJ12A, timlib:SMAJ12A
- U$10: value 2 -> SMAJ12A; device timlib:PWR163 -> timlib:SMAJ12A
- U$9: value 2 -> PSMN1R0-40YSH; device timlib:PWR163 -> timlib:PSMN1R0-40YSH
Connections:
- new net N$2: R1.1, U$11.G, U$12.C
- new net N$3: R5.2, U$9.D
- new net N$4: R4.1, U$10.C, U$9.G
- net GND: now also U$10.A, U$12.A, U$9.S
- net N$1: now also R2.2; no longer U$10.1
Other:
- moved on the sheet: R1
Changed lines of the file:
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@@
 <part name="J7" library="timlib" library_urn="urn:adsk.eagle:library:16152524" deviceset="XT30PW-F" device="" package3d_urn="urn:adsk.eagle:package:16203166/6"/>
 <part name="J8" library="timlib" library_urn="urn:adsk.eagle:library:16152524" deviceset="XT30PW-F" device="" package3d_urn="urn:adsk.eagle:package:16203166/6"/>
-<part name="U$9" library="timlib" library_urn="urn:adsk.eagle:library:16152524" deviceset="PWR163" device="" package3d_urn="urn:adsk.eagle:package:16220013/7" value="2"/>
-<part name="U$10" library="timlib" library_urn="urn:adsk.eagle:library:16152524" deviceset="PWR163" device="" package3d_urn="urn:adsk.eagle:package:16220013/7" value="2"/>
 <part name="U$11" library="timlib" library_urn="urn:adsk.eagle:library:16152524" deviceset="PSMN1R0-40YSH" device="" package3d_urn="urn:adsk.eagle:package:16249927/3"/>
 <part name="GND5" library="supply1" library_urn="urn:adsk.eagle:library:371" deviceset="GND" device=""/>
 <part name="R1" library="rcl" library_urn="urn:adsk.eagle:library:334" deviceset="R-US_" device="R0603" package3d_urn="urn:adsk.eagle:package:23555/3" value="100"/>
+<part name="U$12" library="timlib" library_urn="urn:adsk.eagle:library:16152524" deviceset="SMAJ12A" device="" package3d_urn="urn:adsk.eagle:package:16356227/5"/>
+<part name="R2" library="timlib" library_urn="urn:adsk.eagle:library:16152524" deviceset="PWR163" device="" package3d_urn="urn:adsk.eagle:package:16220013/7" value="2"/>
+<part name="U$9" library="timlib" library_urn="urn:adsk.eagle:library:16152524" deviceset="PSMN1R0-40YSH" device="" package3d_urn="urn:adsk.eagle:package:16249927/3"/>
+<part name="GND6" library="supply1" library_urn="urn:adsk.eagle:library:371" deviceset="GND" device=""/>
+<part name="R4" library="rcl" library_urn="urn:adsk.eagle:library:334" deviceset="R-US_" device="R0603" package3d_urn="urn:adsk.eagle:package:23555/3" value="100"/>
+<part name="U$10" library="timlib" library_urn="urn:adsk.eagle:library:16152524" deviceset="SMAJ12A" device="" package3d_urn="urn:adsk.eagle:package:16356227/5"/>
+<part name="R5" library="timlib" library_urn="urn:adsk.eagle:library:16152524" deviceset="PWR163" device="" package3d_urn="urn:adsk.eagle:package:16220013/7" value="2"/>
 </parts>
 <sheets>
@@
 <attribute name="VALUE" x="155.846" y="138.034" size="1.27" layer="96" font="vector"/>
 </instance>
-<instance part="U$9" gate="G$1" x="215.9" y="104.14" smashed="yes">
-<attribute name="NAME" x="212.09" y="105.6386" size="1.778" layer="95"/>
-<attribute name="VALUE" x="212.09" y="100.838" size="1.778" layer="96"/>
-</instance>
-<instance part="U$10" gate="G$1" x="121.92" y="93.98" smashed="yes" rot="R90">
-<attribute name="NAME" x="120.4214" y="90.17" size="1.778" layer="95" rot="R90"/>
-<attribute name="VALUE" x="125.222" y="90.17" size="1.778" layer="96" rot="R90"/>
-</instance>
 <instance part="U$11" gate="G$1" x="119.38" y="81.28" smashed="yes">
 <attribute name="VALUE" x="107.95" y="85.09" size="1.778" layer="96" rot="MR180"/>
@@
 <attribute name="VALUE" x="119.38" y="66.04" size="1.778" layer="96"/>
 </instance>
-<instance part="R1" gate="G$1" x="106.68" y="91.44" smashed="yes" rot="R90">
-<attribute name="NAME" x="105.1814" y="87.63" size="1.778" layer="95" rot="R90"/>
-<attribute name="VALUE" x="109.982" y="87.63" size="1.778" layer="96" rot="R90"/>
+<instance part="R1" gate="G$1" x="106.68" y="93.98" smashed="yes" rot="R90">
+<attribute name="NAME" x="105.1814" y="90.17" size="1.778" layer="95" rot="R90"/>
+<attribute name="VALUE" x="109.982" y="90.17" size="1.778" layer="96" rot="R90"/>
+</instance>
+<instance part="U$12" gate="G$1" x="111.76" y="73.66" smashed="yes">
+<attribute name="NAME" x="114.554" y="75.565" size="1.778" layer="95"/>
+<attribute name="VALUE" x="114.554" y="72.771" size="1.778" layer="96"/>
+</instance>
+<instance part="R2" gate="G$1" x="121.92" y="93.98" smashed="yes" rot="R270">
+<attribute name="NAME" x="123.4186" y="97.79" size="1.778" layer="95" rot="R270"/>
+<attribute name="VALUE" x="118.618" y="97.79" size="1.778" layer="96" rot="R270"/>
+</instance>
+<instance part="U$9" gate="G$1" x="160.02" y="78.74" smashed="yes">
+<attribute name="VALUE" x="148.59" y="82.55" size="1.778" layer="96" rot="MR180"/>
+<attribute name="NAME" x="148.59" y="80.01" size="1.778" layer="95" rot="MR180"/>
+</instance>
+<instance part="GND6" gate="1" x="162.56" y="66.04" smashed="yes">
+<attribute name="VALUE" x="160.02" y="63.5" size="1.778" layer="96"/>
+</instance>
+<instance part="R4" gate="G$1" x="147.32" y="91.44" smashed="yes" rot="R90">
+<attribute name="NAME" x="145.8214" y="87.63" size="1.778" layer="95" rot="R90"/>
+<attribute name="VALUE" x="150.622" y="87.63" size="1.778" layer="96" rot="R90"/>
+</instance>
+<instance part="U$10" gate="G$1" x="152.4" y="71.12" smashed="yes">
+<attribute name="NAME" x="155.194" y="73.025" size="1.778" layer="95"/>
+<attribute name="VALUE" x="155.194" y="70.231" size="1.778" layer="96"/>
+</instance>
+<instance part="R5" gate="G$1" x="162.56" y="91.44" smashed="yes" rot="R270">
+<attribute name="NAME" x="164.0586" y="95.25" size="1.778" layer="95" rot="R270"/>
+<attribute name="VALUE" x="159.258" y="95.25" size="1.778" layer="96" rot="R270"/>
 </instance>
 </instances>
@@
 <pinref part="GND5" gate="1" pin="GND"/>
 <wire x1="121.92" y1="76.2" x2="121.92" y2="71.12" width="0.1524" layer="91"/>
+<pinref part="U$12" gate="G$1" pin="A"/>
+<wire x1="111.76" y1="71.12" x2="121.92" y2="71.12" width="0.1524" layer="91"/>
+<junction x="121.92" y="71.12"/>
+</segment>
+<segment>
+<pinref part="U$9" gate="G$1" pin="S"/>
+<pinref part="GND6" gate="1" pin="GND"/>
+<wire x1="162.56" y1="73.66" x2="162.56" y2="68.58" width="0.1524" layer="91"/>
+<pinref part="U$10" gate="G$1" pin="A"/>
+<wire x1="152.4" y1="68.58" x2="162.56" y2="68.58" width="0.1524" layer="91"/>
+<junction x="162.56" y="68.58"/>
 </segment>
 </net>
 <net name="N$1" class="0">
 <segment>
-<pinref part="U$10" gate="G$1" pin="1"/>
 <wire x1="121.92" y1="88.9" x2="121.92" y2="86.36" width="0.1524" layer="91"/>
 <pinref part="U$11" gate="G$1" pin="D"/>
-</segment>
-</net>
+<pinref part="R2" gate="G$1" pin="2"/>
+</segment>
+</net>
+<net name="N$2" class="0">
+<segment>
+<pinref part="U$12" gate="G$1" pin="C"/>
+<wire x1="111.76" y1="76.2" x2="111.76" y2="78.74" width="0.1524" layer="91"/>
+<pinref part="U$11" gate="G$1" pin="G"/>
+<wire x1="111.76" y1="78.74" x2="116.84" y2="78.74" width="0.1524" layer="91"/>
+<wire x1="111.76" y1="78.74" x2="106.68" y2="78.74" width="0.1524" layer="91"/>
+<junction x="111.76" y="78.74"/>
+<pinref part="R1" gate="G$1" pin="1"/>
+<wire x1="106.68" y1="78.74" x2="106.68" y2="88.9" width="0.1524" layer="91"/>
+</segment>
+</net>
+<net name="N$3" class="0">
+<segment>
+<wire x1="162.56" y1="86.36" x2="162.56" y2="83.82" width="0.1524" layer="91"/>
+<pinref part="U$9" gate="G$1" pin="D"/>
+<pinref part="R5" gate="G$1" pin="2"/>
+</segment>
+</net>
+<net name="N$4" class="0">
+<segment>
+<pinref part="U$10" gate="G$1" pin="C"/>
+<wire x1="152.4" y1="73.66" x2="152.4" y2="76.2" width="0.1524" layer="91"/>
+<pinref part="U$9" gate="G$1" pin="G"/>
+<wire x1="152.4" y1="76.2" x2="157.48" y2="76.2" width="0.1524" layer="91"/>
+<wire x1="152.4" y1="76.2" x2="147.32" y2="76.2" width="0.1524" layer="91"/>
+<junction x="152.4" y="76.2"/>
+<pinref part="R4" gate="G$1" pin="1"/>
+<wire x1="147.32" y1="76.2" x2="147.32" y2="86.36" width="0.1524" layer="91"/>
+</segment>
+</net>

Commit message: Missing some caps
Parts:
- added C1, C2, C3, C4, C5, C6, C7: 220uf, timlib:35ZLH220MEFC8X11.5
- added IC1, IC2: LM321MF, linear:LM321MF
- added R10, R15, R17, R19, R7, R9: 100k\, rcl:R-US_R0603
- added R11: 4.7k, rcl:R-US_R0603
- added R12: 2, timlib:PWR163
- added R13, R3: 873.1k, rcl:R-US_R0603
- added R14: 100k, rcl:R-US_R0603
- added R16, R18, R6, R8: 400k, rcl:R-US_R0603
- added U$1, U$2, U$3, U$6: PSMN1R0-40YSH, timlib:PSMN1R0-40YSH
- added U$4, U$7, U$8: SMAJ12A, timlib:SMAJ12A
- added U$5: LP2951ACMM/NOPB, timlib:LP2951ACMM/NOPB
- R1: value 100 -> 4.7k
- R4: value 100 -> 100k
- R5: value 2 -> 100k\; device timlib:PWR163 -> rcl:R-US_R0603
- U$9: value PSMN1R0-40YSH -> LP2951ACMM/NOPB; device timlib:PSMN1R0-40YSH -> timlib:LP2951ACMM/NOPB
Connections:
- net GND_12V renamed -12VOUT
- net GND_5V renamed -5VOUT
- net ISO_+12V renamed +12VOUT
- net ISO_+5V renamed +5VOUT
- removed net +24V: J1.PIN1, J5.V+, J6.V+, J7.V+, J8.V+, U1.+VIN, U2.+VIN
- new net BATT_+24V: C1.+, C2.+, C3.+, C4.+, C5.+, C6.+, C7.+, J1.PIN1, J5.V+, J6.V+, J7.V+, J8.V+, U$5.INPUT, U$9.INPUT, U1.+VIN, U2.+VIN
- new net BATT_GND: IC1.V-, IC2.V-, J2.PIN1, R14.1, R16.1, R18.1, R4.1, R6.1, R8.1, U$1.S, U$10.A, U$11.S, U$12.A, U$2.S, U$3.S, U$4.A, U$5.GND, U$5.SHDN, U$8.A, U$9.GND, U$9.SHDN
- new net ISO_12V: IC2.V+, R11.2, R13.2, R15.2, R17.2, U$5.OUT
- new net ISO_GND: R12.2, U$6.D, U1.-VIN, U2.-VIN
- new net LEG_12V: IC1.V+, R1.2, R3.2, R5.2, R7.2, U$9.OUT
- new net LEG_GND: C1.-, C2.-, C3.-, C4.-, C5.-, C6.-, C7.-, J5.V-, J6.V-, J7.V-, J8.V-, R2.1, U$1.D, U$2.D
- new net N$10: R13.1, R14.2, U$5.FEEDB
- new net N$11: R12.1, U$3.D
- new net N$12: IC2.-IN, R15.1, R16.2
- new net N$13: IC2.+IN, R17.1, R18.2
- new net N$14: IC2.OUT, R19.2
- new net N$15: R19.1, U$6.G, U$7.C
- new net N$5: IC1.+IN, R7.1, R8.2
- new net N$6: IC1.OUT, R10.2, R9.2
- new net N$7: R11.1, U$3.G, U$4.C
- new net N$8: R9.1, U$1.G, U$8.C
- new net N$9: R10.1, U$10.C, U$2.G
- net GND: now also U$6.S, U$7.A; no longer J2.PIN1, J5.V-, J6.V-, J7.V-, J8.V-, U$10.A, U$11.S, U$12.A, U$9.S, U1.-VIN, U2.-VIN
- net N$3: now also R3.1, R4.2, U$9.FEEDB; no longer R5.2, U$9.D
- net N$4: now also IC1.-IN, R5.1, R6.2; no longer R4.1, U$10.C, U$9.G
Other:
- note added: "PWR RESIST"
- moved on the sheet: J3, J4, J5, J6, J7, J8, R1, R2, R4, R5, U$10, U$11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

Commit message: More caps
Parts:
- removed U$10, U$12, U$4, U$7, U$8: SMAJ12A, timlib:SMAJ12A
- added C10, C11, C8, C9: 2.2uF, timlib:C0402
- added C12, C13: 300nF, timlib:C0402
- added D1, D2, D3, D4, D5: SMAJ12A, timlib:SMAJ12A
- added R20, R21: 0.5, rcl:R-US_R0603
- R18, R8: value 400k -> 500k
Connections:
- new net BATT_+24V1: C10.1
- new net N$16: C9.1, R20.1
- new net N$17: C11.1, R21.1
- net BATT_+24V: now also C8.1
- net BATT_GND: now also D2.A, D3.A, D4.A, D5.A; no longer U$10.A, U$12.A, U$4.A, U$8.A
- net GND: now also C10.2, C11.2, C12.2, C13.2, C8.2, C9.2, D1.A; no longer U$7.A
- net ISO_12V: now also R20.2
- net LEG_12V: now also R21.2
- net N$13: now also C13.1
- net N$15: now also D1.C; no longer U$7.C
- net N$2: now also D4.C; no longer U$12.C
- net N$5: now also C12.1
- net N$7: now also D5.C; no longer U$4.C
- net N$8: now also D3.C; no longer U$8.C
- net N$9: now also D2.C; no longer U$10.C
Other:
- moved on the sheet: IC1, IC2, R1, R10, R11, R12, R15, R16, R17, R18, R19, R2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

Commit message: More updates to power board
Parts:
- added U$26, U$27: 2-PIN, timlib:2-PIN
- added U$4: CDBB5100-HF, timlib:CDBB5100-HF
- R10, R19, R9: value 100k\ -> 4.7k
Connections:
- removed net -12VOUT: J3.CONN1, J3.CONN3, U2.-VOUT
- removed net -5VOUT: J4.CONN1, J4.CONN3, U1.-VOUT
- removed net BATT_+24V: C1.+, C2.+, C3.+, C4.+, C5.+, C6.+, C7.+, C8.1, J1.PIN1, J5.V+, J6.V+, J7.V+, J8.V+, U$5.INPUT, U$9.INPUT, U1.+VIN, U2.+VIN
- removed net BATT_+24V1: C10.1
- removed net GND: C10.2, C11.2, C12.2, C13.2, C8.2, C9.2, D1.A, U$6.S
- new net +24V: C1.+, C2.+, C3.+, C4.+, C5.+, C6.+, C7.+, J1.PIN1, J5.V+, J6.V+, J7.V+, J8.V+, U$26.P$1, U$27.P$1, U$4.C, U1.+VIN, U2.+VIN
- new net 12V_GND: J3.CONN1, J3.CONN3, U2.12V_GND
- new net 5V_GND: J4.CONN1, J4.CONN3, U1.5V_GND
- new net N$18: C8.1, U$26.P$2, U$5.INPUT
- new net N$19: C10.1, U$27.P$2, U$9.INPUT
- net +12VOUT: now also U2.+12VOUT; no longer U2.+VOUT
- net +5VOUT: now also U1.+5VOUT; no longer U1.+VOUT
- net BATT_GND: now also C10.2, C11.2, C12.2, C13.2, C8.2, C9.2, D1.A, U$6.S
- net LEG_GND: now also U$4.A
Other:
- note added: "SWITCH"
- moved on the sheet: C10, C11, C12, D2, D3, D4, IC1, J5, J6, J7, J8, R1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

Commit message: part moving
Parts:
- C10, C11, C12, C13, C8, C9: device timlib:C0402 -> timlib:C_CERAMIC_0603
Other:
- moved on the sheet: C10, C11, C12, C13, C8, C9, D1, D2, D3, D4, D5, IC1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

Commit message: Updates to power board
Parts:
- J1, J2: value FASTON_MALE_RA_BLADE -> FASTON1289_ST; device timlib:FASTON_MALE_RA_BLADE -> timlib:FASTON1289_ST
Other:
- moved on the sheet: R2
Changed lines of the file:
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@@
 </variantdefs>
 <classes>
-<class number="0" name="default" width="0" drill="0">
+<class number="0" name="default" width="0" drill="0.3">
 </class>
-<class number="1" name="High current" width="0.762" drill="0">
+<class number="1" name="power plane" width="0" drill="0">
+<clearance class="1" value="0.5"/>
+</class>
+<class number="2" name="power via" width="0" drill="0.25">
+<clearance class="2" value="0.0254"/>
 </class>
 </classes>
@@
 <parts>
 <part name="FRAME1" library="frames" library_urn="urn:adsk.eagle:library:229" deviceset="FRAME_A_L" device=""/>
-<part name="J1" library="timlib" library_urn="urn:adsk.eagle:library:16152524" deviceset="FASTON_MALE_RA_BLADE" device="" package3d_urn="urn:adsk.eagle:package:16188667/3"/>
-<part name="J2" library="timlib" library_urn="urn:adsk.eagle:library:16152524" deviceset="FASTON_MALE_RA_BLADE" device="" package3d_urn="urn:adsk.eagle:package:16188667/3"/>
+<part name="J1" library="timlib" library_urn="urn:adsk.eagle:library:16152524" deviceset="FASTON" device="1289_ST" package3d_urn="urn:adsk.eagle:package:16406409/2"/>
+<part name="J2" library="timlib" library_urn="urn:adsk.eagle:library:16152524" deviceset="FASTON" device="1289_ST" package3d_urn="urn:adsk.eagle:package:16406409/2"/>
 <part name="P+1" library="timlib" library_urn="urn:adsk.eagle:library:16152524" deviceset="V_BATT" device=""/>
 <part name="J3" library="timlib" library_urn="urn:adsk.eagle:library:16152524" deviceset="MOLEX_4_RA" device="" package3d_urn="urn:adsk.eagle:package:16152611/3" value="12v"/>
@@
 <attribute name="VALUE" x="87.122" y="59.69" size="1.778" layer="96" rot="R90"/>
 </instance>
-<instance part="R2" gate="G$1" x="106.68" y="83.82" smashed="yes" rot="R180" grouprefs="LEG_SOFTSTART">
-<attribute name="NAME" x="105.41" y="87.4014" size="1.778" layer="95" rot="R180"/>
-<attribute name="VALUE" x="105.41" y="82.042" size="1.778" layer="96" rot="R180"/>
+<instance part="R2" gate="G$1" x="106.68" y="83.82" smashed="yes" grouprefs="LEG_SOFTSTART">
+<attribute name="NAME" x="107.95" y="80.2386" size="1.778" layer="95"/>
+<attribute name="VALUE" x="107.95" y="85.598" size="1.778" layer="96"/>
 </instance>
 <instance part="U$9" gate="G$1" x="45.72" y="78.74" smashed="yes" rot="R180" grouprefs="LEG_SOFTSTART">
@@
 <pinref part="R2" gate="G$1" pin="1"/>
 <pinref part="U$1" gate="G$1" pin="D"/>
-<wire x1="111.76" y1="83.82" x2="170.18" y2="83.82" width="0.1524" layer="91" grouprefs="LEG_SOFTSTART"/>
+<wire x1="101.6" y1="83.82" x2="170.18" y2="83.82" width="0.1524" layer="91" grouprefs="LEG_SOFTSTART"/>
 <wire x1="170.18" y1="83.82" x2="170.18" y2="73.66" width="0.1524" layer="91" grouprefs="LEG_SOFTSTART"/>
 <pinref part="U$2" gate="G$1" pin="D"/>
@@
 </segment>
 </net>
-<net name="ISO_GND" class="0">
+<net name="ISO_GND" class="1">
 <segment>
 <pinref part="U2" gate="G$1" pin="-VIN"/>
@@
 <pinref part="R12" gate="G$1" pin="2"/>
 <wire x1="170.18" y1="160.02" x2="170.18" y2="165.1" width="0.1524" layer="91" grouprefs="ISO_SOFTSTART"/>
-<wire x1="114.3" y1="160.02" x2="170.18" y2="160.02" width="0.1524" layer="91" grouprefs="ISO_SOFTSTART"/>
-<junction x="170.18" y="160.02" grouprefs="ISO_SOFTSTART"/>
+<wire x1="114.3" y1="160.02" x2="170.18" y2="160.02" width="0.1524" layer="91"/>
+<junction x="170.18" y="160.02"/>
 </segment>
 </net>
@@
 <pinref part="R2" gate="G$1" pin="2"/>
 <wire x1="99.06" y1="60.96" x2="99.06" y2="83.82" width="0.1524" layer="91" grouprefs="LEG_SOFTSTART"/>
-<wire x1="99.06" y1="83.82" x2="101.6" y2="83.82" width="0.1524" layer="91" grouprefs="LEG_SOFTSTART"/>
+<wire x1="99.06" y1="83.82" x2="111.76" y2="83.82" width="0.1524" layer="91" grouprefs="LEG_SOFTSTART"/>
 </segment>
 </net>
@@
 </segment>
 </net>
-<net name="N$11" class="0">
-<segment>
-<pinref part="R12" gate="G$1" pin="1"/>
-<wire x1="104.14" y1="160.02" x2="101.6" y2="160.02" width="0.1524" layer="91" grouprefs="ISO_SOFTSTART"/>
-<pinref part="U$3" gate="G$1" pin="D"/>
-<wire x1="101.6" y1="160.02" x2="101.6" y2="137.16" width="0.1524" layer="91" grouprefs="ISO_SOFTSTART"/>
-</segment>
-</net>
-<net name="+24V" class="1">
+<net name="+24V" class="0">
 <segment>
 <pinref part="U2" gate="G$1" pin="+VIN"/>
@@
 </segment>
 </net>
-<net name="N$18" class="1">
+<net name="N$18" class="0">
 <segment>
 <pinref part="U$5" gate="G$1" pin="INPUT"/>
@@
 </segment>
 </net>
-<net name="N$19" class="1">
+<net name="N$19" class="0">
 <segment>
 <pinref part="U$9" gate="G$1" pin="INPUT"/>
@@
 </segment>
 </net>
+<net name="N$11" class="1">
+<segment>
+<pinref part="U$3" gate="G$1" pin="D"/>
+<wire x1="101.6" y1="137.16" x2="101.6" y2="160.02" width="0.1524" layer="91"/>
+<pinref part="R12" gate="G$1" pin="1"/>
+<wire x1="101.6" y1="160.02" x2="104.14" y2="160.02" width="0.1524" layer="91"/>
+</segment>
+</net>
