File: hardware/power/power_board.sch (EAGLE design)
At the start: 61 parts, among them IC1 LM321MF, IC2 LM321MF, J1 FASTON1289_ST, J2 FASTON1289_ST, J3 12v, J4 5v, J5 XT30PW-F, J6 XT30PW-F, J7 XT30PW-F, J8 XT30PW-F, U1 PDQ30-Q24-S5-D, U2 PDQ30-Q24-S12-D

Commit message: First power plane layout attempt
Connections:
- net +24V renamed BATT_+24V
Changed lines of the file:
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@@
 <parts>
 <part name="FRAME1" library="frames" library_urn="urn:adsk.eagle:library:229" deviceset="FRAME_A_L" device=""/>
-<part name="J1" library="timlib" library_urn="urn:adsk.eagle:library:16152524" deviceset="FASTON" device="1289_ST" package3d_urn="urn:adsk.eagle:package:16406409/2"/>
-<part name="J2" library="timlib" library_urn="urn:adsk.eagle:library:16152524" deviceset="FASTON" device="1289_ST" package3d_urn="urn:adsk.eagle:package:16406409/2"/>
+<part name="J1" library="timlib" library_urn="urn:adsk.eagle:library:16152524" deviceset="FASTON" device="1289_ST" package3d_urn="urn:adsk.eagle:package:16406409/3"/>
+<part name="J2" library="timlib" library_urn="urn:adsk.eagle:library:16152524" deviceset="FASTON" device="1289_ST" package3d_urn="urn:adsk.eagle:package:16406409/3"/>
 <part name="P+1" library="timlib" library_urn="urn:adsk.eagle:library:16152524" deviceset="V_BATT" device=""/>
 <part name="J3" library="timlib" library_urn="urn:adsk.eagle:library:16152524" deviceset="MOLEX_4_RA" device="" package3d_urn="urn:adsk.eagle:package:16152611/3" value="12v"/>
 <part name="J4" library="timlib" library_urn="urn:adsk.eagle:library:16152524" deviceset="MOLEX_4_RA" device="" package3d_urn="urn:adsk.eagle:package:16152611/3" value="5v"/>
-<part name="U1" library="timlib" library_urn="urn:adsk.eagle:library:16152524" deviceset="PDQ30-Q24-S5-D" device="" package3d_urn="urn:adsk.eagle:package:16187995/2"/>
-<part name="U2" library="timlib" library_urn="urn:adsk.eagle:library:16152524" deviceset="PDQ30-Q24-S12-D" device="" package3d_urn="urn:adsk.eagle:package:16187995/2"/>
+<part name="U1" library="timlib" library_urn="urn:adsk.eagle:library:16152524" deviceset="PDQ30-Q24-S5-D" device="" package3d_urn="urn:adsk.eagle:package:16187995/3"/>
+<part name="U2" library="timlib" library_urn="urn:adsk.eagle:library:16152524" deviceset="PDQ30-Q24-S12-D" device="" package3d_urn="urn:adsk.eagle:package:16187995/3"/>
 <part name="J5" library="timlib" library_urn="urn:adsk.eagle:library:16152524" deviceset="XT30PW-F" device="" package3d_urn="urn:adsk.eagle:package:16203166/6"/>
 <part name="J6" library="timlib" library_urn="urn:adsk.eagle:library:16152524" deviceset="XT30PW-F" device="" package3d_urn="urn:adsk.eagle:package:16203166/6"/>
 <part name="J7" library="timlib" library_urn="urn:adsk.eagle:library:16152524" deviceset="XT30PW-F" device="" package3d_urn="urn:adsk.eagle:package:16203166/6"/>
 <part name="J8" library="timlib" library_urn="urn:adsk.eagle:library:16152524" deviceset="XT30PW-F" device="" package3d_urn="urn:adsk.eagle:package:16203166/6"/>
-<part name="U$11" library="timlib" library_urn="urn:adsk.eagle:library:16152524" deviceset="PSMN1R0-40YSH" device="" package3d_urn="urn:adsk.eagle:package:16249927/3"/>
+<part name="U$11" library="timlib" library_urn="urn:adsk.eagle:library:16152524" deviceset="PSMN1R0-40YSH" device="" package3d_urn="urn:adsk.eagle:package:16249927/4"/>
 <part name="R1" library="rcl" library_urn="urn:adsk.eagle:library:334" deviceset="R-US_" device="R0603" package3d_urn="urn:adsk.eagle:package:23555/3" value="4.7k"/>
-<part name="R2" library="timlib" library_urn="urn:adsk.eagle:library:16152524" deviceset="PWR163" device="" package3d_urn="urn:adsk.eagle:package:16220013/7" value="2"/>
+<part name="R2" library="timlib" library_urn="urn:adsk.eagle:library:16152524" deviceset="PWR163" device="" package3d_urn="urn:adsk.eagle:package:16220013/8" value="2"/>
 <part name="U$9" library="timlib" library_urn="urn:adsk.eagle:library:16152524" deviceset="LP2951ACMM/NOPB" device="" package3d_urn="urn:adsk.eagle:package:16380727/2"/>
 <part name="R3" library="rcl" library_urn="urn:adsk.eagle:library:334" deviceset="R-US_" device="R0603" package3d_urn="urn:adsk.eagle:package:23555/3" value="873.1k"/>
@@
 <part name="R7" library="rcl" library_urn="urn:adsk.eagle:library:334" deviceset="R-US_" device="R0603" package3d_urn="urn:adsk.eagle:package:23555/3" value="100k\"/>
 <part name="R8" library="rcl" library_urn="urn:adsk.eagle:library:334" deviceset="R-US_" device="R0603" package3d_urn="urn:adsk.eagle:package:23555/3" value="500k"/>
-<part name="U$1" library="timlib" library_urn="urn:adsk.eagle:library:16152524" deviceset="PSMN1R0-40YSH" device="" package3d_urn="urn:adsk.eagle:package:16249927/3"/>
-<part name="U$2" library="timlib" library_urn="urn:adsk.eagle:library:16152524" deviceset="PSMN1R0-40YSH" device="" package3d_urn="urn:adsk.eagle:package:16249927/3"/>
+<part name="U$1" library="timlib" library_urn="urn:adsk.eagle:library:16152524" deviceset="PSMN1R0-40YSH" device="" package3d_urn="urn:adsk.eagle:package:16249927/4"/>
+<part name="U$2" library="timlib" library_urn="urn:adsk.eagle:library:16152524" deviceset="PSMN1R0-40YSH" device="" package3d_urn="urn:adsk.eagle:package:16249927/4"/>
 <part name="R9" library="rcl" library_urn="urn:adsk.eagle:library:334" deviceset="R-US_" device="R0603" package3d_urn="urn:adsk.eagle:package:23555/3" value="4.7k"/>
 <part name="R10" library="rcl" library_urn="urn:adsk.eagle:library:334" deviceset="R-US_" device="R0603" package3d_urn="urn:adsk.eagle:package:23555/3" value="4.7k"/>
-<part name="U$3" library="timlib" library_urn="urn:adsk.eagle:library:16152524" deviceset="PSMN1R0-40YSH" device="" package3d_urn="urn:adsk.eagle:package:16249927/3"/>
+<part name="U$3" library="timlib" library_urn="urn:adsk.eagle:library:16152524" deviceset="PSMN1R0-40YSH" device="" package3d_urn="urn:adsk.eagle:package:16249927/4"/>
 <part name="R11" library="rcl" library_urn="urn:adsk.eagle:library:334" deviceset="R-US_" device="R0603" package3d_urn="urn:adsk.eagle:package:23555/3" value="4.7k"/>
-<part name="R12" library="timlib" library_urn="urn:adsk.eagle:library:16152524" deviceset="PWR163" device="" package3d_urn="urn:adsk.eagle:package:16220013/7" value="2"/>
+<part name="R12" library="timlib" library_urn="urn:adsk.eagle:library:16152524" deviceset="PWR163" device="" package3d_urn="urn:adsk.eagle:package:16220013/8" value="2"/>
 <part name="U$5" library="timlib" library_urn="urn:adsk.eagle:library:16152524" deviceset="LP2951ACMM/NOPB" device="" package3d_urn="urn:adsk.eagle:package:16380727/2"/>
 <part name="R13" library="rcl" library_urn="urn:adsk.eagle:library:334" deviceset="R-US_" device="R0603" package3d_urn="urn:adsk.eagle:package:23555/3" value="873.1k"/>
@@
 <part name="R17" library="rcl" library_urn="urn:adsk.eagle:library:334" deviceset="R-US_" device="R0603" package3d_urn="urn:adsk.eagle:package:23555/3" value="100k\"/>
 <part name="R18" library="rcl" library_urn="urn:adsk.eagle:library:334" deviceset="R-US_" device="R0603" package3d_urn="urn:adsk.eagle:package:23555/3" value="500k"/>
-<part name="U$6" library="timlib" library_urn="urn:adsk.eagle:library:16152524" deviceset="PSMN1R0-40YSH" device="" package3d_urn="urn:adsk.eagle:package:16249927/3"/>
+<part name="U$6" library="timlib" library_urn="urn:adsk.eagle:library:16152524" deviceset="PSMN1R0-40YSH" device="" package3d_urn="urn:adsk.eagle:package:16249927/4"/>
 <part name="R19" library="rcl" library_urn="urn:adsk.eagle:library:334" deviceset="R-US_" device="R0603" package3d_urn="urn:adsk.eagle:package:23555/3" value="4.7k"/>
 <part name="R20" library="rcl" library_urn="urn:adsk.eagle:library:334" deviceset="R-US_" device="R0603" package3d_urn="urn:adsk.eagle:package:23555/3" value="0.5"/>
@@
 </segment>
 </net>
-<net name="LEG_GND" class="0">
+<net name="LEG_GND" class="1">
 <segment>
 <pinref part="J8" gate="G$1" pin="V-"/>
@@
 </segment>
 </net>
-<net name="+5VOUT" class="0">
+<net name="+5VOUT" class="1">
 <segment>
 <pinref part="U1" gate="G$1" pin="+5VOUT"/>
@@
 </segment>
 </net>
-<net name="+12VOUT" class="0">
+<net name="+12VOUT" class="1">
 <segment>
 <pinref part="J3" gate="G$1" pin="CONN4"/>
@@
 </segment>
 </net>
-<net name="+24V" class="0">
+<net name="BATT_+24V" class="1">
 <segment>
 <pinref part="U2" gate="G$1" pin="+VIN"/>
@@
 </segment>
 </net>
-<net name="5V_GND" class="0">
+<net name="5V_GND" class="1">
 <segment>
 <pinref part="J4" gate="G$1" pin="CONN1"/>
@@
 </segment>
 </net>
-<net name="12V_GND" class="0">
+<net name="12V_GND" class="1">
 <segment>
 <pinref part="J3" gate="G$1" pin="CONN3"/>
