File: hardware/power/power_board.sch (EAGLE design)
At the start: 61 parts, among them IC1 LM321MF, IC2 LM321MF, J1 FASTON1289_ST, J2 FASTON1289_ST, J3 12v, J4 5v, J5 XT30PW-F, J6 XT30PW-F, J7 XT30PW-F, J8 XT30PW-F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

Commit message: REVERT TO EARLIER
Parts:
- removed U$4: CDBB5100-HF, timlib:CDBB5100-HF
- added C14, C15, C16, C17, C18, C19, C20, C21, C22, C23: 10uF, timlib:C_CERAMIC_1210
- added D6, D7: SK510A-LTP, timlib:SK510A-LTP
Connections:
- net BATT_+24V: now also C14.1, C15.1, C16.1, C17.1, C18.1, C19.1, C20.1, C21.1, C22.1, C23.1, D6.C, D7.C; no longer U$4.C
- net ISO_GND: now also C14.2, C15.2, C16.2, C17.2, C18.2, C19.2, C20.2, C21.2, C22.2, C23.2
- net LEG_GND: now also D6.A, D7.A; no longer U$4.A
Other:
- moved on the sheet: R2
