File: hardware/power/power_board.brd (EAGLE design)
At the start: 92 x 92 mm, 61 parts, among them IC1 LM321MF, IC2 LM321MF, J1 FASTON1289_ST, J2 FASTON1289_ST, J3 12v, J4 5v, J5 XT30PW-F, J6 XT30PW-F, J7 XT30PW-F, J8 XT30PW-F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

Commit message: REVERT TO EARLIER
Parts:
- removed U$4: CDBB5100-HF, timlib:DO-214AA
- added C14, C15, C16, C17, C18, C19, C20, C21, C22, C23: 10uF, timlib:C1210
- added D6, D7: SK510A-LTP, timlib:DO-214AC
- moved D2 23.3 mm to (43.8, 36.6)
- moved U$2 23.3 mm to (35.7, 36.8)
- moved R10 23.0 mm to (46.6, 36.9)
- moved U$11 22.0 mm to (35.9, 58.5)
- moved D4 21.8 mm to (41.1, 58.5)
- moved R1 21.8 mm to (44.1, 58.5)
- moved U$26 5.00 mm to (58.9, 10.7)
- moved U$27 5.00 mm to (68.8, 10.7)
- moved C13 4.47 mm to (44.9, 16.4), turned to 270 degrees
- moved C1 4.27 mm to (14.7, 24.0), turned to 90 degrees
- moved C12 4.06 mm to (45.0, 26.4), turned to 270 degrees
- moved U$1 3.15 mm to (36.0, 52.4)
- moved R2 3.00 mm to (36.0, 44.4)
- moved D1 2.40 mm to (23.7, 10.9)
- moved D5 2.40 mm to (23.7, 4.50)
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Connections:
- net BATT_+24V: now also C14.1, C15.1, C16.1, C17.1, C18.1, C19.1, C20.1, C21.1, C22.1, C23.1, D6.C, D7.C; no longer U$4.C
- net ISO_GND: now also C14.2, C15.2, C16.2, C17.2, C18.2, C19.2, C20.2, C21.2, C22.2, C23.2
- net LEG_GND: now also D6.A, D7.A; no longer U$4.A
Routing:
- net BATT_GND: track 45.5 -> 75.2 mm
- net BATT_+24V: track 3.72 -> 33.0 mm, vias 0 -> 1
- net LEG_12V: track 27.5 -> 53.2 mm
- net N$6: track 43.7 -> 57.7 mm
- net ISO_12V: track 46.9 -> 57.1 mm
- net N$13: track 19.1 -> 27.2 mm
- net N$5: track 18.8 -> 25.5 mm
- net N$8: track 11.6 -> 5.97 mm
- net ISO_GND: track 0.00 -> 5.23 mm, vias 0 -> 98
- net N$18: track 22.1 -> 26.6 mm
- net N$14: track 22.5 -> 26.5 mm
- net N$2: track 10.3 -> 6.42 mm
- net N$3: track 15.1 -> 18.3 mm
- net N$12: track 13.9 -> 16.5 mm
- net N$10: track 15.0 -> 17.5 mm
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- added copper zone on layer 1, net BATT_+24V
- added copper zone on layer 16, net ISO_GND

Commit message: Fixed weird export issue
Parts:
- moved D2 23.0 mm to (44.0, 59.5)
- moved U$2 22.8 mm to (34.5, 59.5)
- moved R10 22.7 mm to (47.0, 59.5)
- moved D4 22.2 mm to (44.0, 36.5)
- moved R1 22.2 mm to (47.0, 36.5)
- moved U$11 22.1 mm to (34.5, 36.5)
- moved U$26 5.00 mm to (53.9, 10.7)
- moved U$27 5.00 mm to (63.9, 10.7)
- moved C13 4.47 mm to (48.5, 18.9), turned to 180 degrees
- moved C12 4.06 mm to (48.4, 28.6), turned to 180 degrees
- moved R9 3.03 mm to (47.0, 51.9), turned to 90 degrees
- moved D3 2.87 mm to (44.0, 51.9)
- moved D1 2.40 mm to (26.1, 10.9)
- moved D5 2.40 mm to (26.1, 4.50)
- moved IC2 2.04 mm to (48.4, 14.4)
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Routing:
- net LEG_12V: track 53.2 -> 26.5 mm
- net BATT_GND: track 75.2 -> 53.0 mm
- net N$6: track 57.7 -> 43.7 mm
- net ISO_12V: track 57.1 -> 46.9 mm
- net N$13: track 27.2 -> 19.1 mm
- net N$5: track 25.5 -> 18.8 mm
- net N$8: track 5.97 -> 11.6 mm
- net N$18: track 26.6 -> 22.1 mm
- net N$14: track 26.5 -> 22.5 mm
- net N$2: track 6.42 -> 10.3 mm
- net N$3: track 18.3 -> 15.1 mm
- net N$12: track 16.5 -> 13.9 mm
- net N$10: track 17.5 -> 15.0 mm
- net N$15: track 11.0 -> 9.09 mm
- net N$9: track 8.71 -> 10.3 mm
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