File: hardware/power/power_board.brd (EAGLE design)
At the start: 92 x 92 mm, 72 parts, among them IC1 LM321MF, IC2 LM321MF, J1 FASTON1289_ST, J2 FASTON1289_ST, J3 12v, J4 5v, J5 XT30PW-F, J6 XT30PW-F, J7 XT30PW-F, J8 XT30PW-F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

Commit message: Added LEDs:
Parts:
- added D10: LTST-C191KRKT, timlib:LTST-C191TBKT
- added D8, D9: LTST-C191TBKT, timlib:LTST-C191TBKT
- added R22, R23, R24: 470, rcl:R0603
Connections:
- new net N$20: D9.A, R22.1
- new net N$21: D8.A, R23.1
- new net N$22: D10.A, R24.1
- net +12VOUT: now also R22.2
- net +5VOUT: now also R23.2
- net 12V_GND: now also D9.C
- net 5V_GND: now also D8.C
- net BATT_+24V: now also R24.2
- net LEG_GND: now also D10.C
Routing:
- net BATT_+24V: track 33.0 -> 36.1 mm
- net N$21: track 0.00 -> 3.04 mm
- net N$20: track 0.00 -> 2.89 mm
- net 5V_GND: track 93.7 -> 95.9 mm
- net 12V_GND: track 76.9 -> 79.0 mm
- net +12VOUT: track 86.6 -> 88.8 mm
- net +5VOUT: track 81.6 -> 83.7 mm
- net N$22: track 0.00 -> 1.81 mm
Changed lines of the file:
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@@
 <element name="U1" library="timlib" library_urn="urn:adsk.eagle:library:16152524" package="PDQ30-D" package3d_urn="urn:adsk.eagle:package:16187995/3" value="PDQ30-Q24-S5-D" x="13.8" y="46.05" smashed="yes" rot="R180"/>
 <element name="U2" library="timlib" library_urn="urn:adsk.eagle:library:16152524" package="PDQ30-D" package3d_urn="urn:adsk.eagle:package:16187995/3" value="PDQ30-Q24-S12-D" x="13.8" y="71.85" smashed="yes"/>
-<element name="J5" library="timlib" library_urn="urn:adsk.eagle:library:16152524" package="XT30PW-F" package3d_urn="urn:adsk.eagle:package:16203166/7" value="XT30PW-F" x="80.85" y="27.333" smashed="yes" rot="R270" grouprefs="EXTERNAL_PLUGS LEG_POWER"/>
-<element name="J6" library="timlib" library_urn="urn:adsk.eagle:library:16152524" package="XT30PW-F" package3d_urn="urn:adsk.eagle:package:16203166/7" value="XT30PW-F" x="80.85" y="41.067" smashed="yes" rot="R270" grouprefs="EXTERNAL_PLUGS LEG_POWER"/>
-<element name="J7" library="timlib" library_urn="urn:adsk.eagle:library:16152524" package="XT30PW-F" package3d_urn="urn:adsk.eagle:package:16203166/7" value="XT30PW-F" x="80.85" y="54.8" smashed="yes" rot="R270" grouprefs="EXTERNAL_PLUGS LEG_POWER"/>
-<element name="J8" library="timlib" library_urn="urn:adsk.eagle:library:16152524" package="XT30PW-F" package3d_urn="urn:adsk.eagle:package:16203166/7" value="XT30PW-F" x="80.85" y="13.6" smashed="yes" rot="R270" grouprefs="EXTERNAL_PLUGS LEG_POWER"/>
+<element name="J5" library="timlib" library_urn="urn:adsk.eagle:library:16152524" package="XT30PW-F" package3d_urn="urn:adsk.eagle:package:16203166/7" value="XT30PW-F" x="80.85" y="27.333" smashed="yes" rot="R270" grouprefs="LEG_POWER EXTERNAL_PLUGS"/>
+<element name="J6" library="timlib" library_urn="urn:adsk.eagle:library:16152524" package="XT30PW-F" package3d_urn="urn:adsk.eagle:package:16203166/7" value="XT30PW-F" x="80.85" y="41.067" smashed="yes" rot="R270" grouprefs="LEG_POWER EXTERNAL_PLUGS"/>
+<element name="J7" library="timlib" library_urn="urn:adsk.eagle:library:16152524" package="XT30PW-F" package3d_urn="urn:adsk.eagle:package:16203166/7" value="XT30PW-F" x="80.85" y="54.8" smashed="yes" rot="R270" grouprefs="LEG_POWER EXTERNAL_PLUGS"/>
+<element name="J8" library="timlib" library_urn="urn:adsk.eagle:library:16152524" package="XT30PW-F" package3d_urn="urn:adsk.eagle:package:16203166/7" value="XT30PW-F" x="80.85" y="13.6" smashed="yes" rot="R270" grouprefs="LEG_POWER EXTERNAL_PLUGS"/>
 <element name="U$11" library="timlib" library_urn="urn:adsk.eagle:library:16152524" package="LFPAK56E" package3d_urn="urn:adsk.eagle:package:16249927/4" value="PSMN1R0-40YSH" x="34.5" y="36.45" smashed="yes" rot="R90" grouprefs="LEG_SOFTSTART"/>
 <element name="R1" library="rcl" library_urn="urn:adsk.eagle:library:334" package="R0603" package3d_urn="urn:adsk.eagle:package:23555/3" value="4.7k" x="46.95" y="36.45" smashed="yes" rot="R270" grouprefs="LEG_SOFTSTART">
@@
 <element name="D6" library="timlib" library_urn="urn:adsk.eagle:library:16152524" package="DO-214AC" package3d_urn="urn:adsk.eagle:package:16356227/6" value="SK510A-LTP" x="77.85" y="3.9" smashed="yes"/>
 <element name="D7" library="timlib" library_urn="urn:adsk.eagle:library:16152524" package="DO-214AC" package3d_urn="urn:adsk.eagle:package:16356227/6" value="SK510A-LTP" x="72.15" y="50.25" smashed="yes" rot="R270"/>
+<element name="R22" library="rcl" library_urn="urn:adsk.eagle:library:334" package="R0603" package3d_urn="urn:adsk.eagle:package:23555/3" value="470" x="75" y="78.3" smashed="yes">
+<attribute name="NAME" x="74.365" y="78.935" size="1.27" layer="25"/>
+<attribute name="POPULARITY" value="77" x="75" y="78.3" size="1.778" layer="27" display="off"/>
+<attribute name="SPICEPREFIX" value="R" x="75" y="78.3" size="1.778" layer="27" display="off"/>
+<attribute name="VALUE" x="74.365" y="76.395" size="1.27" layer="27"/>
+</element>
+<element name="R23" library="rcl" library_urn="urn:adsk.eagle:library:334" package="R0603" package3d_urn="urn:adsk.eagle:package:23555/3" value="470" x="75" y="67.05" smashed="yes">
+<attribute name="NAME" x="74.365" y="67.685" size="1.27" layer="25"/>
+<attribute name="POPULARITY" value="77" x="75" y="67.05" size="1.778" layer="27" display="off"/>
+<attribute name="SPICEPREFIX" value="R" x="75" y="67.05" size="1.778" layer="27" display="off"/>
+<attribute name="VALUE" x="74.365" y="65.145" size="1.27" layer="27"/>
+</element>
+<element name="D8" library="timlib" library_urn="urn:adsk.eagle:library:16152524" package="LTST-C191TBKT" package3d_urn="urn:adsk.eagle:package:16446604/3" value="LTST-C191TBKT" x="75" y="70.05" smashed="yes" rot="R180">
+<attribute name="NAME" x="76.5" y="69.05" size="1.27" layer="25" rot="R180"/>
+<attribute name="VALUE" x="76.5" y="72.25" size="1.27" layer="27" rot="R180"/>
+</element>
+<element name="D9" library="timlib" library_urn="urn:adsk.eagle:library:16152524" package="LTST-C191TBKT" package3d_urn="urn:adsk.eagle:package:16446604/3" value="LTST-C191TBKT" x="75" y="81.15" smashed="yes" rot="R180">
+<attribute name="NAME" x="76.5" y="80.15" size="1.27" layer="25" rot="R180"/>
+<attribute name="VALUE" x="76.5" y="83.35" size="1.27" layer="27" rot="R180"/>
+</element>
+<element name="D10" library="timlib" library_urn="urn:adsk.eagle:library:16152524" package="LTST-C191TBKT" package3d_urn="urn:adsk.eagle:package:16446604/3" value="LTST-C191KRKT" x="73.2" y="5.85" smashed="yes" rot="R90">
+<attribute name="NAME" x="72.2" y="4.35" size="1.27" layer="25" rot="R90"/>
+<attribute name="VALUE" x="75.4" y="4.35" size="1.27" layer="27" rot="R90"/>
+</element>
+<element name="R24" library="rcl" library_urn="urn:adsk.eagle:library:334" package="R0603" package3d_urn="urn:adsk.eagle:package:23555/3" value="470" x="74.1" y="8.4" smashed="yes">
+<attribute name="NAME" x="73.465" y="9.035" size="1.27" layer="25"/>
+<attribute name="POPULARITY" value="77" x="74.1" y="8.4" size="1.778" layer="27" display="off"/>
+<attribute name="SPICEPREFIX" value="R" x="74.1" y="8.4" size="1.778" layer="27" display="off"/>
+<attribute name="VALUE" x="73.465" y="6.495" size="1.27" layer="27"/>
+</element>
 </elements>
 <signals>
@@
 <vertex x="70.65" y="1.232353125"/>
 </polygon>
+<contactref element="D10" pad="C"/>
 </signal>
 <signal name="ISO_GND" class="1">
@@
 <wire x1="21.45" y1="67.3" x2="21.45" y2="58.72" width="2" layer="1"/>
 <wire x1="21.45" y1="58.72" x2="23.96" y2="56.21" width="2" layer="1"/>
+<contactref element="R23" pad="2"/>
+<wire x1="75.85" y1="67.05" x2="77.78" y2="67.05" width="0.1524" layer="1"/>
+<wire x1="77.78" y1="67.05" x2="77.88" y2="66.95" width="0.1524" layer="1"/>
 </signal>
 <signal name="+12VOUT" class="1">
@@
 <wire x1="14.25" y1="72.3" x2="3.64" y2="61.69" width="2" layer="1"/>
 <wire x1="74.2444625" y1="81.2" x2="30.2855375" y2="81.2" width="2" layer="16"/>
+<contactref element="R22" pad="2"/>
+<wire x1="75.85" y1="78.3" x2="77.68" y2="78.3" width="0.1524" layer="1"/>
+<wire x1="77.68" y1="78.3" x2="77.88" y2="78.1" width="0.1524" layer="1"/>
 </signal>
 <signal name="N$7">
@@
 <wire x1="15.493" y1="89.6" x2="18" y2="89.6" width="2" layer="1"/>
 <wire x1="11.26" y1="85.367" x2="15.493" y2="89.6" width="2" layer="1"/>
+<contactref element="R24" pad="2"/>
+<wire x1="74.95" y1="8.4" x2="74.95" y2="10.2" width="0.1524" layer="1"/>
+<wire x1="74.95" y1="10.2" x2="75.85" y2="11.1" width="0.1524" layer="1"/>
 </signal>
 <signal name="5V_GND" class="1">
@@
 <wire x1="31.3855375" y1="78.7" x2="73.208925" y2="78.7" width="2" layer="16"/>
 <wire x1="80.88" y1="69.95" x2="77.88" y2="69.95" width="2" layer="16"/>
+<contactref element="D8" pad="C"/>
+<wire x1="75.76" y1="70.05" x2="77.78" y2="70.05" width="0.1524" layer="1"/>
+<wire x1="77.78" y1="70.05" x2="77.88" y2="69.95" width="0.1524" layer="1"/>
 </signal>
 <signal name="12V_GND" class="1">
@@
 <wire x1="24" y1="61.73" x2="23.96" y2="61.69" width="2" layer="1"/>
 <wire x1="75.28" y1="83.7" x2="29.25" y2="83.7" width="2" layer="16"/>
+<contactref element="D9" pad="C"/>
+<wire x1="75.76" y1="81.15" x2="77.83" y2="81.15" width="0.1524" layer="1"/>
+<wire x1="77.83" y1="81.15" x2="77.88" y2="81.1" width="0.1524" layer="1"/>
 </signal>
 <signal name="N$18">
@@
 </polygon>
 </signal>
+<signal name="N$20">
+<contactref element="R22" pad="1"/>
+<contactref element="D9" pad="A"/>
+<wire x1="74.24" y1="81.15" x2="74.24" y2="78.39" width="0.1524" layer="1"/>
+<wire x1="74.24" y1="78.39" x2="74.15" y2="78.3" width="0.1524" layer="1"/>
+</signal>
+<signal name="N$21">
+<contactref element="R23" pad="1"/>
+<contactref element="D8" pad="A"/>
+<wire x1="74.24" y1="70.05" x2="74.15" y2="69.96" width="0.1524" layer="1"/>
+<wire x1="74.15" y1="69.96" x2="74.15" y2="67.05" width="0.1524" layer="1"/>
+</signal>
+<signal name="N$22">
+<contactref element="D10" pad="A"/>
+<contactref element="R24" pad="1"/>
+<wire x1="73.2" y1="6.61" x2="73.2" y2="8.35" width="0.1524" layer="1"/>
+<wire x1="73.2" y1="8.35" x2="73.25" y2="8.4" width="0.1524" layer="1"/>
+</signal>
 </signals>
