File: hardware/power/power_v3.sch (EAGLE design)
At the start: 32 parts, among them J1 LINEAR_2_5040500291, J2 PWR_2_XT30PW-F, J3 PWR_2_XT30PW-F, J4 PWR_2_XT30PW-F, J5 PWR_2_XT30PW-F, Q1 CSD19536KTT, U1 PDQ30-Q24-S5-D, U2 PDQ30-Q24-S12-D, U3 LM5069

Commit message: Spinning IC
Parts:
- added C12: 0.068uF 50V, _T_rcl:C0603
- added C13: 0.012uF 50V, _T_rcl:C0603
- added D3: SCHOTTKY_SOD123, _T_rcl:SCHOTTKY_SOD123
- added D4: D, _T_rcl:D
- added J10: LINEAR_2_5040500291, _T_conn:LINEAR_2_5040500291
- added J6, J7: FASTON, _T_power:FASTON
- added J8, J9: PWR_4, _T_conn:PWR_4
- added Q2: CSD19536KTT, _T_transistors:CSD19536KTT
- added R10: 20k, _T_rcl:R0603
- added R11: 2.4, _T_rcl:R0603
- added R12: 10, _T_rcl:R0603
- added R13: 47k 1%, _T_rcl:R0603
- added R14: 2.7k 1%, _T_rcl:R0603
- added R15: 4.7k 1%, _T_rcl:R0603
- added R16: 1k, _T_rcl:R0603
- added R9: .002, _T_rcl:R_SENSE_2512
- added U4: LM5069, _T_ic:LM5069
Connections:
- new net N$14: Q2.D, R9.2
- new net N$15: C12.1, U4.TIMER
- new net N$16: R10.2, U4.PWR
- new net N$17: R11.1, R12.1, U4.SEN
- new net N$18: R11.2, R9.K2
- new net N$19: R13.1, R14.2, U4.UVLO
- new net N$20: R14.1, R15.2, U4.OVLO
- new net N$21: J10.P1, R13.2
- new net N$22: R12.2, R9.K1
- new net N$23: C13.1, D4.C
- new net N$24: D4.A, Q2.G, R16.2, U4.GATE
- net +12V: now also J9.P2, J9.P4
- net +24V_ISO: now also D3.C, Q2.S, U4.OUT
- net +5V: now also J8.P2, J8.P4
- net +V_BATT: now also J10.P2, J6.PIN1, R9.1, U4.VIN
- net -V_BATT: now also C12.2, C13.2, D3.A, J7.PIN1, R10.1, R15.1, R16.1, U4.GND
- net 12V_GND: now also J9.P1, J9.P3
- net 5V_GND: now also J8.P1, J8.P3
Other:
- moved on the sheet: C10, C11, L1, L2, U1, U2

Commit message: TVS diodes
Parts:
- added C14: 0.068uF 50V, _T_rcl:C0603
- added D5: 5_0SMDJ24A, _T_rcl:SCHOTTKY_SOD123
- D1, D3: value SCHOTTKY_SOD123 -> 5_0SMDJ24A
- D2: value D -> (none)
- D4: value D -> 1N4148W-7-F
Connections:
- net +V_BATT: now also C14.1, D5.C
- net -V_BATT: now also C14.2, D5.A
Changed lines of the file:
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@@
 <part name="R1" library="_T_rcl" library_urn="urn:adsk.eagle:library:19571919" deviceset="R_SENSE" device="_2512" package3d_urn="urn:adsk.eagle:package:21272979/2" value=".002"/>
 <part name="Q1" library="_T_transistors" library_urn="urn:adsk.eagle:library:19605452" deviceset="CSD19536KTT" device="" package3d_urn="urn:adsk.eagle:package:21297419/2"/>
-<part name="D1" library="_T_rcl" library_urn="urn:adsk.eagle:library:19571919" deviceset="SCHOTTKY" device="_SOD123" package3d_urn="urn:adsk.eagle:package:20295471/2"/>
+<part name="D1" library="_T_rcl" library_urn="urn:adsk.eagle:library:19571919" deviceset="SCHOTTKY" device="_SOD123" package3d_urn="urn:adsk.eagle:package:20295471/2" value="5_0SMDJ24A"/>
 <part name="GND7" library="_T_power" library_urn="urn:adsk.eagle:library:19572085" deviceset="-V_BATT" device=""/>
 <part name="C1" library="_T_rcl" library_urn="urn:adsk.eagle:library:19571919" deviceset="C" device="0603" package3d_urn="urn:adsk.eagle:package:19572011/3" value="0.068uF 50V"/>
@@
 <part name="R9" library="_T_rcl" library_urn="urn:adsk.eagle:library:19571919" deviceset="R_SENSE" device="_2512" package3d_urn="urn:adsk.eagle:package:21272979/2" value=".002"/>
 <part name="Q2" library="_T_transistors" library_urn="urn:adsk.eagle:library:19605452" deviceset="CSD19536KTT" device="" package3d_urn="urn:adsk.eagle:package:21297419/2"/>
-<part name="D3" library="_T_rcl" library_urn="urn:adsk.eagle:library:19571919" deviceset="SCHOTTKY" device="_SOD123" package3d_urn="urn:adsk.eagle:package:20295471/2"/>
+<part name="D3" library="_T_rcl" library_urn="urn:adsk.eagle:library:19571919" deviceset="SCHOTTKY" device="_SOD123" package3d_urn="urn:adsk.eagle:package:20295471/2" value="5_0SMDJ24A"/>
 <part name="GND5" library="_T_power" library_urn="urn:adsk.eagle:library:19572085" deviceset="-V_BATT" device=""/>
 <part name="C12" library="_T_rcl" library_urn="urn:adsk.eagle:library:19571919" deviceset="C" device="0603" package3d_urn="urn:adsk.eagle:package:19572011/3" value="0.068uF 50V"/>
@@
 <part name="GND11" library="_T_power" library_urn="urn:adsk.eagle:library:19572085" deviceset="-V_BATT" device=""/>
 <part name="J10" library="_T_conn" library_urn="urn:adsk.eagle:library:19570503" deviceset="LINEAR_2" device="_5040500291" package3d_urn="urn:adsk.eagle:package:20672635/2"/>
-<part name="D4" library="_T_rcl" library_urn="urn:adsk.eagle:library:19571919" deviceset="D" device="" package3d_urn="urn:adsk.eagle:package:20295471/2"/>
+<part name="D4" library="_T_rcl" library_urn="urn:adsk.eagle:library:19571919" deviceset="D" device="" package3d_urn="urn:adsk.eagle:package:20295471/2" value="1N4148W-7-F"/>
 <part name="R16" library="_T_rcl" library_urn="urn:adsk.eagle:library:19571919" deviceset="R" device="0603" package3d_urn="urn:adsk.eagle:package:19572012/3" value="1k"/>
 <part name="C13" library="_T_rcl" library_urn="urn:adsk.eagle:library:19571919" deviceset="C" device="0603" package3d_urn="urn:adsk.eagle:package:19572011/3" value="0.012uF 50V"/>
 <part name="GND12" library="_T_power" library_urn="urn:adsk.eagle:library:19572085" deviceset="-V_BATT" device=""/>
+<part name="C14" library="_T_rcl" library_urn="urn:adsk.eagle:library:19571919" deviceset="C" device="0603" package3d_urn="urn:adsk.eagle:package:19572011/3" value="0.068uF 50V"/>
+<part name="D5" library="_T_rcl" library_urn="urn:adsk.eagle:library:19571919" deviceset="SCHOTTKY" device="_SOD123" package3d_urn="urn:adsk.eagle:package:20295471/2" value="5_0SMDJ24A"/>
 </parts>
 <sheets>
@@
 <attribute name="VALUE" x="23.876" y="178.689" size="1.778" layer="96"/>
 </instance>
-<instance part="J6" gate="G$1" x="142.24" y="187.96" smashed="yes" grouprefs="BATT_TERM"/>
+<instance part="J6" gate="G$1" x="142.24" y="190.5" smashed="yes" grouprefs="BATT_TERM"/>
 <instance part="J7" gate="G$1" x="142.24" y="182.88" smashed="yes" grouprefs="BATT_TERM"/>
 <instance part="J8" gate="G$1" x="91.44" y="182.88" smashed="yes" grouprefs="5V_ISO">
@@
 <instance part="GND12" gate="G$1" x="119.38" y="-7.62" smashed="yes" grouprefs="+ISO_POWER">
 <attribute name="VALUE" x="117.475" y="-10.795" size="1.778" layer="96"/>
+</instance>
+<instance part="C14" gate="G$1" x="132.08" y="187.96" smashed="yes">
+<attribute name="NAME" x="133.604" y="188.341" size="1.778" layer="95"/>
+<attribute name="VALUE" x="133.604" y="183.261" size="1.778" layer="96"/>
+</instance>
+<instance part="D5" gate="G$1" x="137.16" y="185.42" smashed="yes" rot="R90">
+<attribute name="NAME" x="135.255" y="183.134" size="1.778" layer="95" rot="R90"/>
 </instance>
 </instances>
@@
 <segment>
 <pinref part="J6" gate="G$1" pin="PIN1"/>
-<wire x1="139.7" y1="187.96" x2="137.16" y2="187.96" width="0.1524" layer="91" grouprefs="BATT_TERM"/>
-<label x="137.16" y="187.96" size="1.778" layer="95" rot="R180" xref="yes" grouprefs="BATT_TERM"/>
+<label x="124.46" y="190.5" size="1.778" layer="95" rot="R180" xref="yes" grouprefs="BATT_TERM"/>
+<wire x1="139.7" y1="190.5" x2="137.16" y2="190.5" width="0.1524" layer="91" grouprefs="BATT_TERM"/>
+<pinref part="C14" gate="G$1" pin="1"/>
+<wire x1="137.16" y1="190.5" x2="132.08" y2="190.5" width="0.1524" layer="91" grouprefs="BATT_TERM"/>
+<wire x1="132.08" y1="190.5" x2="124.46" y2="190.5" width="0.1524" layer="91" grouprefs="BATT_TERM"/>
+<junction x="132.08" y="190.5"/>
+<pinref part="D5" gate="G$1" pin="C"/>
+<wire x1="137.16" y1="187.96" x2="137.16" y2="190.5" width="0.1524" layer="91"/>
+<junction x="137.16" y="190.5"/>
 </segment>
 <segment>
@@
 <segment>
 <pinref part="J7" gate="G$1" pin="PIN1"/>
+<label x="124.46" y="182.88" size="1.778" layer="95" rot="R180" xref="yes" grouprefs="BATT_TERM"/>
 <wire x1="139.7" y1="182.88" x2="137.16" y2="182.88" width="0.1524" layer="91" grouprefs="BATT_TERM"/>
-<label x="137.16" y="182.88" size="1.778" layer="95" rot="R180" xref="yes" grouprefs="BATT_TERM"/>
-</segment>
-<segment>
+<pinref part="C14" gate="G$1" pin="2"/>
+<wire x1="137.16" y1="182.88" x2="132.08" y2="182.88" width="0.1524" layer="91" grouprefs="BATT_TERM"/>
+<wire x1="132.08" y1="182.88" x2="124.46" y2="182.88" width="0.1524" layer="91" grouprefs="BATT_TERM"/>
+<junction x="132.08" y="182.88"/>
+<pinref part="D5" gate="G$1" pin="A"/>
+<junction x="137.16" y="182.88"/>
+</segment>
+<segment>

Commit message: Ready to PCB it
Parts:
- D2: value (none) -> 1N4148W-7-F
Changed lines of the file:
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@@
 <part name="J4" library="_T_conn" library_urn="urn:adsk.eagle:library:19570503" deviceset="PWR_2" device="_XT30PW-F" package3d_urn="urn:adsk.eagle:package:20295843/2"/>
 <part name="J5" library="_T_conn" library_urn="urn:adsk.eagle:library:19570503" deviceset="PWR_2" device="_XT30PW-F" package3d_urn="urn:adsk.eagle:package:20295843/2"/>
-<part name="D2" library="_T_rcl" library_urn="urn:adsk.eagle:library:19571919" deviceset="D" device="" package3d_urn="urn:adsk.eagle:package:20295471/2"/>
+<part name="D2" library="_T_rcl" library_urn="urn:adsk.eagle:library:19571919" deviceset="D" device="" package3d_urn="urn:adsk.eagle:package:20295471/2" value="1N4148W-7-F"/>
 <part name="R8" library="_T_rcl" library_urn="urn:adsk.eagle:library:19571919" deviceset="R" device="0603" package3d_urn="urn:adsk.eagle:package:19572012/3" value="1k"/>
 <part name="C2" library="_T_rcl" library_urn="urn:adsk.eagle:library:19571919" deviceset="C" device="0603" package3d_urn="urn:adsk.eagle:package:19572011/3" value="0.012uF 50V"/>
