File: hardware/ahrs/ahrs.sch (EAGLE design)
At the start: 6 parts, among them U1 LSM9DS1

Commit message: Updates to AHRS
Parts:
- added C10, C11, C13, C15, C8, C9: 100nF, rcl:C-EUC0603
- added C12: 4.7uF, rcl:C-EUC0603
- added C14: 1uFnet, rcl:C-EUC0603
- added C16, C17: 6.2pF, rcl:C-EUC0603
- added C6: 10nF, rcl:C-EUC0603
- added C7: 1uF, rcl:C-EUC0603
- added L1: 600R@100MHz, timlib:CHOKE
- added U2: STM32G4_UFQFPN48_T1, timlib:STM32G4_UFQFPN48_T1
- added X1: NX2016SA24MHZ-EXS00A-CS11335, timlib:NX2016SA24MHZ-EXS00A-CS11335
Connections:
- new net N$1: C6.1, C7.1, U2B.VDDA
- new net N$5: C17.1, U2A.PF1-OSC_OUT, X1.1
- new net N$6: C16.1, U2A.PF0-OSC_IN, X1.2
- new net VREF: C13.1, C14.1, L1.2, U2B.VREF+
- net GND: now also C10.2, C11.2, C12.2, C13.2, C14.2, C15.2, C16.2, C17.2, C6.2, C7.2, C8.2, C9.2, U2B.EPAD, X1.GND
- net VDD: now also C10.1, C11.1, C12.1, C15.1, C8.1, C9.1, L1.1, U2B.VBAT, U2B.VDD, U2B.VDD_2, U2B.VDD_3

Commit message: More AHRS updates
Parts:
- added C18, C19: 1uF 10v, rcl:C-EUC0603
- added C20, C21: 22uF 10v, rcl:C-EUC0603
- added U$1: LDFM33PUR, timlib:LDFM33PUR
- added U$3: MCP2542FD, timlib:MCP2542FD
- C1, C10, C11, C13, C15, C3, C5, C8, C9: value 100nF -> 100nF 10v
- C12: value 4.7uF -> 4.7uF 10v
- C14: value 1uFnet -> 1uF 10v
- C16, C17: value 6.2pF -> 6.2pF 10v
- C2: value 10uF -> 10uF 10v
- C4: value 10nF(>=16V) -> 10nF 16v
- C6: value 10nF -> 100nF 10v
- C7: value 1uF -> 1uF 10v
Connections:
- new net 5V: C19.1, U$1.EN, U$1.VIN
- new net CAN_RX: U$3.RXD, U2A.PA11
- new net CAN_TX: U$3.TXD, U2A.PA12
- new net CS_AG: U1.CS_A/G
- new net CS_M: U1.CS_M
- new net INT1_AG: U1.INT1_A/G, U2A.PB0
- new net INT2_AG: U1.INT2_A/G, U2A.PC4
- new net INT_M: U1.INT_M, U2A.PB1
- new net LPUART1_TX: U2A.PA2
- new net MISO: U1.SDO_A/G, U1.SDO_M, U2A.PA6
- new net MOSI: U1.SDA/SDI/SDO, U2A.PA7
- new net NRST: U2A.PG10-NRST
- new net SCK: U1.SCL/SPC, U2A.PA5
- net GND: now also C18.2, C19.2, C20.2, C21.2, U$1.GND
- net VDD: now also C18.1, C20.1, C21.1, U$1.VOUT
Other:
- moved on the sheet: U2A

Commit message: Laying out ahrs
Parts:
- removed C8: 100nF 10v, rcl:C-EUC0603
- added C22, C23: 0.1uF 10v, rcl:C-EUC0603
- added D1: SMAJ5A, timlib:SMAJ5A
- added J1: 2-PIN, timlib:2-PIN
- added U$5: 3-PIN, timlib:3-PIN
- added X2: SM08B-SRSS-TB, con-jst2:SM08B-SRSS-TB
Connections:
- removed net LPUART1_TX: U2A.PA2
- removed net VDD: C10.1, C11.1, C12.1, C15.1, C18.1, C2.1, C20.1, C21.1, C3.1, C5.1, C8.1, C9.1, L1.1, U$1.VOUT, U1.VDD@1, U1.VDD@2, U2B.VBAT, U2B.VDD, U2B.VDD_2, U2B.VDD_3
- new net 3.3V: C10.1, C11.1, C12.1, C15.1, C18.1, C2.1, C20.1, C21.1, C22.1, C3.1, C5.1, C9.1, L1.1, U$1.VOUT, U$3.VIO, U1.VDD@1, U1.VDD@2, U2B.VBAT, U2B.VDD, U2B.VDD_2, U2B.VDD_3, X2-1.S
- new net CAN_H: U$3.CANH, U$5.P$2
- new net CAN_L: U$3.CANL, U$5.P$1
- new net LPUART_RX: U2A.PB10, X2-8.S
- new net LPUART_TX: U2A.PA2, X2-3.S
- new net SWCLK: U2A.PA14, X2-5.S
- new net SWDIO: U2A.PA13, X2-4.S
- new net SWO: U2A.PB3, X2-6.S
- net 5V: now also C23.1, D1.C, J1.P$1, U$3.VDD
- net CS_AG: now also U2A.PA3
- net CS_M: now also U2A.PA4
- net GND: now also C22.2, C23.2, D1.A, J1.P$2, U$3.VSS, U$5.P$3, U2A.PB8-BOOT0, X2-2.S; no longer C8.2
- net NRST: now also X2-7.S
Other:
- moved on the sheet: C16, C17, X1

Commit message: R1 of ahrs
Other:
- moved on the sheet: C1, C10, C11, C12, C13, C14, C15, C16, C17, C18, C19, C2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

Commit message: Prior to pulling from fusion
Parts:
- C1, C2, C3, C4, C5: device timlib:C_CERAMIC_0603 -> rcl:C-EUC0603
- X2: device con-jst2:SM08B-SRSS-TB -> timlib:SM08B-SRSS-TB
Changed lines of the file:
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@@
 <?xml version="1.0" encoding="utf-8"?>
 <!DOCTYPE eagle SYSTEM "eagle.dtd">
-<eagle version="9.5.2">
+<eagle version="9.6.1">
 <drawing>
 <settings>
@@
 <part name="FRAME1" library="frames" library_urn="urn:adsk.eagle:library:229" deviceset="FRAME_A_L" device=""/>
 <part name="U1" library="timlib" library_urn="urn:adsk.eagle:library:16152524" deviceset="LSM9DS1" device="" package3d_urn="urn:adsk.eagle:package:18130566/2"/>
-<part name="C1" library="timlib" library_urn="urn:adsk.eagle:library:16152524" deviceset="C_CERAMIC" device="_0603" package3d_urn="urn:adsk.eagle:package:23616/2" value="100nF 10v"/>
+<part name="C1" library="rcl" library_urn="urn:adsk.eagle:library:334" deviceset="C-EU" device="C0603" package3d_urn="urn:adsk.eagle:package:23616/2" value="100nF 10v"/>
 <part name="GND1" library="supply1" library_urn="urn:adsk.eagle:library:371" deviceset="GND" device=""/>
 <part name="VDD1" library="supply1" library_urn="urn:adsk.eagle:library:371" deviceset="VDD" device=""/>
 <part name="GND2" library="supply1" library_urn="urn:adsk.eagle:library:371" deviceset="GND" device=""/>
-<part name="C2" library="timlib" library_urn="urn:adsk.eagle:library:16152524" deviceset="C_CERAMIC" device="_0603" package3d_urn="urn:adsk.eagle:package:23616/2" value="10uF 10v"/>
-<part name="C3" library="timlib" library_urn="urn:adsk.eagle:library:16152524" deviceset="C_CERAMIC" device="_0603" package3d_urn="urn:adsk.eagle:package:23616/2" value="100nF 10v"/>
-<part name="C4" library="timlib" library_urn="urn:adsk.eagle:library:16152524" deviceset="C_CERAMIC" device="_0603" package3d_urn="urn:adsk.eagle:package:23616/2" value="10nF 16v"/>
+<part name="C2" library="rcl" library_urn="urn:adsk.eagle:library:334" deviceset="C-EU" device="C0603" package3d_urn="urn:adsk.eagle:package:23616/2" override_package3d_urn="urn:adsk.eagle:package:19477979/2" override_package_urn="urn:adsk.eagle:footprint:23123/1" value="10uF 10v"/>
+<part name="C3" library="rcl" library_urn="urn:adsk.eagle:library:334" deviceset="C-EU" device="C0603" package3d_urn="urn:adsk.eagle:package:23616/2" value="100nF 10v"/>
+<part name="C4" library="rcl" library_urn="urn:adsk.eagle:library:334" deviceset="C-EU" device="C0603" package3d_urn="urn:adsk.eagle:package:23616/2" value="10nF 16v"/>
 <part name="GND4" library="supply1" library_urn="urn:adsk.eagle:library:371" deviceset="GND" device=""/>
 <part name="VDD2" library="supply1" library_urn="urn:adsk.eagle:library:371" deviceset="VDD" device=""/>
-<part name="C5" library="timlib" library_urn="urn:adsk.eagle:library:16152524" deviceset="C_CERAMIC" device="_0603" package3d_urn="urn:adsk.eagle:package:23616/2" value="100nF 10v"/>
+<part name="C5" library="rcl" library_urn="urn:adsk.eagle:library:334" deviceset="C-EU" device="C0603" package3d_urn="urn:adsk.eagle:package:23616/2" value="100nF 10v"/>
 <part name="FRAME2" library="frames" library_urn="urn:adsk.eagle:library:229" deviceset="FRAME_A_L" device=""/>
-<part name="U2" library="timlib" library_urn="urn:adsk.eagle:library:16152524" deviceset="STM32G4_UFQFPN48_T1" device="" package3d_urn="urn:adsk.eagle:package:19324073/1"/>
+<part name="U2" library="timlib" library_urn="urn:adsk.eagle:library:16152524" deviceset="STM32G4_UFQFPN48_T1" device="" package3d_urn="urn:adsk.eagle:package:19324073/1" override_package3d_urn="urn:adsk.eagle:package:19324073/2" override_package_urn="urn:adsk.eagle:footprint:19324070/1"/>
 <part name="C6" library="rcl" library_urn="urn:adsk.eagle:library:334" deviceset="C-EU" device="C0603" package3d_urn="urn:adsk.eagle:package:23616/2" value="100nF 10v"/>
 <part name="C7" library="rcl" library_urn="urn:adsk.eagle:library:334" deviceset="C-EU" device="C0603" package3d_urn="urn:adsk.eagle:package:23616/2" value="1uF 10v"/>
@@
 <part name="U$5" library="timlib" library_urn="urn:adsk.eagle:library:16152524" deviceset="3-PIN" device="" package3d_urn="urn:adsk.eagle:package:16399489/2"/>
 <part name="GND15" library="supply1" library_urn="urn:adsk.eagle:library:371" deviceset="GND" device=""/>
-<part name="X2" library="con-jst2" library_urn="urn:adsk.eagle:library:19399826" deviceset="?M08B-SRSS-TB" device="S" package3d_urn="urn:adsk.eagle:package:19399895/1"/>
+<part name="X2" library="timlib" library_urn="urn:adsk.eagle:library:16152524" deviceset="?M08B-SRSS-TB" device="S" package3d_urn="urn:adsk.eagle:package:19399895/3"/>
 <part name="J1" library="timlib" library_urn="urn:adsk.eagle:library:16152524" deviceset="2-PIN" device="" package3d_urn="urn:adsk.eagle:package:16399492/4"/>
 <part name="GND16" library="supply1" library_urn="urn:adsk.eagle:library:371" deviceset="GND" device=""/>
@@
 will not be understood (or retained) with this version.
 </note>
+<note version="9.4" severity="warning">
+Since Version 9.4, EAGLE supports the overriding of 3D packages
+in schematics and board files. Those overridden 3d packages
+will not be understood (or retained) with this version.
+</note>

Commit message: Rerouting much better
Connections:
- net N$1 renamed VDDA
Changed lines of the file:
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@@
 <class number="0" name="default" width="0" drill="0">
+</class>
+<class number="1" name="power" width="0.3" drill="0">
 </class>
 </classes>
@@
 </busses>
 <nets>
-<net name="GND" class="0">
+<net name="GND" class="1">
 <segment>
 <pinref part="C1" gate="G$1" pin="1"/>
@@
 </segment>
 </net>
-<net name="3.3V" class="0">
+<net name="3.3V" class="1">
 <segment>
 <pinref part="U1" gate="G$1" pin="VDD@1"/>
@@
 </segment>
 </net>
-<net name="N$1" class="0">
+<net name="VDDA" class="1">
 <segment>
 <pinref part="C7" gate="G$1" pin="1"/>
@@
 </segment>
 </net>
-<net name="VREF" class="0">
+<net name="VREF" class="1">
 <segment>
 <pinref part="C14" gate="G$1" pin="1"/>
@@
 </segment>
 </net>
-<net name="5V" class="0">
+<net name="5V" class="1">
 <segment>
 <pinref part="U$1" gate="G$1" pin="VIN"/>

Commit message: Pre logo
Parts:
- removed U$5: 3-PIN, timlib:3-PIN
- added D2: LED_0603150060RS75000, timlib:LED_0603150060RS75000
- added H1, H2, H3, H4: GND_HOLE_M3, timlib:GND_HOLE_M3
- added J2: 3-PIN3, timlib:3-PIN3
- added R1: 68, rcl:R-US_R0603
- renumbered U$1 to U3, U$3 to U4, X2 to J3
Connections:
- new net N$1: D2.C, R1.2
- net 3.3V: now also D2.A
- net CAN_H: now also J2.P$2; no longer U$5.P$2
- net CAN_L: now also J2.P$1; no longer U$5.P$1
- net GND: now also H1.GND_HOLE, H2.GND_HOLE, H3.GND_HOLE, H4.GND_HOLE, J2.P$3, R1.1; no longer U$5.P$3
