File: hardware/ahrs/ahrs.sch (EAGLE design)
At the start: 38 parts, among them J1 2-PIN, J2 3-PIN3, J3 SM08B-SRSS-TB, U1 LSM9DS1, U2 STM32G4_UFQFPN48_T1, U3 LDFM33PUR, U4 MCP2542FD, X1 NX2016SA24MHZ-EXS00A-CS11335

Commit message: Added LEDs and updates for PCBway
Parts:
- added D3, D4: LED_0603150060RS75000, timlib:LED_0603150060RS75000
- added R2, R3: 68, rcl:R-US_R0603
- J1: value 2-PIN -> LINEAR_2_JST_SH_RA; device timlib:2-PIN -> _T_conn:LINEAR_2_JST_SH_RA
- J2: value 3-PIN3 -> LINEAR_3_JST_PH_RA; device timlib:3-PIN3 -> _T_conn:LINEAR_3_JST_PH_RA
- J3: value SM08B-SRSS-TB -> LINEAR_8_JST_PH_RA; device timlib:SM08B-SRSS-TB -> _T_conn:LINEAR_8_JST_PH_RA
Connections:
- new net N$10: R3.1, U2A.PB15
- new net N$7: R2.1, U2A.PB14
- new net N$8: D3.A, R2.2
- new net N$9: D4.A, R3.2
- net 3.3V: now also J3.P1; no longer J3-1.S
- net 5V: now also J1.P1; no longer J1.P$1
- net CAN_H: now also J2.P2; no longer J2.P$2
- net CAN_L: now also J2.P1; no longer J2.P$1
- net GND: now also D3.C, D4.C, J1.P2, J2.P3, J3.P2; no longer J1.P$2, J2.P$3, J3-2.S
- net LPUART_RX: now also J3.P8; no longer J3-8.S
- net LPUART_TX: now also J3.P3; no longer J3-3.S
- net NRST: now also J3.P7; no longer J3-7.S
- net SWCLK: now also J3.P5; no longer J3-5.S
- net SWDIO: now also J3.P4; no longer J3-4.S
- net SWO: now also J3.P6; no longer J3-6.S

Commit message: POSSIBLY BAD MERGE
Parts:
- removed H1, H2, H3, H4: GND_HOLE_M3, timlib:GND_HOLE_M3
- removed J2: LINEAR_3_JST_PH_RA, _T_conn:LINEAR_3_JST_PH_RA
- added C8: 0.1uF 10V, _T_rcl:C0603
- added J4: LINEAR_35040500391, _T_conn:LINEAR_35040500391
- added L2: 600R@100MHz, _T_rcl:DC_CHOKE_FERRITE_BEAD_0603
- added R4: (no value), _T_rcl:R0603
- C1, C10, C13, C15, C3, C5, C6, C9: value 100nF 10v -> 0.1uF 10V; device rcl:C-EUC0603 -> _T_rcl:C0603
- C11, C12, C14, C18, C19, C2, C22, C23, C4, C7: device rcl:C-EUC0603 -> _T_rcl:C0603
- C16, C17: value 6.2pF 10v -> 10pF 10v; device rcl:C-EUC0603 -> _T_rcl:C0603
- C20, C21: value 22uF 10v -> 2.2uF 10V; device rcl:C-EUC0603 -> _T_rcl:C0603
- D1: value SMAJ5A -> (none); device timlib:SMAJ5A -> _T_rcl:TVS_SOD123
- D2, D3, D4: value LED_0603150060RS75000 -> 150060BS75000; device timlib:LED_0603150060RS75000 -> _T_rcl:LED_0603
- J1: value LINEAR_2_JST_SH_RA -> LINEAR_2_5040500291; device _T_conn:LINEAR_2_JST_SH_RA -> _T_conn:LINEAR_2_5040500291
- J3: value LINEAR_8_JST_PH_RA -> LINEAR_85040500891; device _T_conn:LINEAR_8_JST_PH_RA -> _T_conn:LINEAR_85040500891
- L1: device timlib:CHOKE -> _T_rcl:DC_CHOKE_FERRITE_BEAD_0603
- R1, R2, R3: value 68 -> 22; device rcl:R-US_R0603 -> _T_rcl:R0603
- U1: device timlib:LSM9DS1 -> _T_ic:LSM9DS1
- U2: device timlib:STM32G4_UFQFPN48_T1 -> _T_ic:STM32G4_UFQFPN48_T1
- U3: device timlib:LDFM33PUR -> _T_ic:LDFM33PUR
- U4: device timlib:MCP2542FD -> _T_ic:MCP2542FD
- X1: value NX2016SA24MHZ-EXS00A-CS11335 -> CRYSTAL_NX2016SA-24MHZ-EXS00A-CS11335; device timlib:NX2016SA24MHZ-EXS00A-CS11335 -> _T_ic:CRYSTAL_NX2016SA-24MHZ-EXS00A-CS11335
Connections:
- net 5V renamed +5V
- removed net 3.3V: C10.1, C11.1, C12.1, C15.1, C18.1, C2.1, C20.1, C21.1, C22.1, C3.1, C5.1, C9.1, D2.A, J3.P1, L1.1, U1.VDD@1, U1.VDD@2, U2B.VBAT, U2B.VDD, U2B.VDD_2, U2B.VDD_3, U3.VOUT, U4.VIO
- removed net CAN_H: J2.P2, U4.CANH
- removed net CAN_L: J2.P1, U4.CANL
- removed net INT1_AG: U1.INT1_A/G, U2A.PB0
- removed net INT2_AG: U1.INT2_A/G, U2A.PC4
- removed net INT_M: U1.INT_M, U2A.PB1
- new net +3V3: C10.1, C11.1, C12.1, C15.1, C18.1, C2.1, C20.1, C21.1, C22.1, C3.1, C5.1, C8.1, C9.1, D2.A, J3.P1, L1.1, L2.2, U1.VDD@1, U1.VDD@2, U2B.VBAT, U2B.VDD, U2B.VDD_2, U2B.VDD_3, U3.VOUT, U4.VIO
- new net N$11: J4.P1, R4.2, U4.CANH
- new net N$12: J4.P2, R4.1, U4.CANL
- net GND: now also C8.2, J4.P3, R2.2, R3.2, U4.STBY; no longer D3.C, D4.C, H1.GND_HOLE, H2.GND_HOLE, H3.GND_HOLE, H4.GND_HOLE, J2.P3
- net N$10: now also D4.C; no longer U2A.PB15
- net N$7: now also D4.A, U2A.PB15; no longer R2.1, U2A.PB14
- net N$8: now also U2A.PB13; no longer R2.2
- net N$9: now also D3.C, R2.1; no longer D4.A, R3.2
- net VDDA: now also L2.1
Other:
- moved on the sheet: C10, C11, C12, C22, C23, C9, D3, D4, J1, J3, R2, R3

Commit message: Initial Power v3
Parts:
- C2: value 10uF 10v -> 10uF 10V
Changed lines of the file:
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@@
 <part name="C1" library="_T_rcl" library_urn="urn:adsk.eagle:library:19571919" deviceset="C" device="0603" package3d_urn="urn:adsk.eagle:package:19572011/3" value="0.1uF 10V"/>
 <part name="VDD1" library="_T_power" library_urn="urn:adsk.eagle:library:19572085" deviceset="+3V3" device=""/>
-<part name="C2" library="_T_rcl" library_urn="urn:adsk.eagle:library:19571919" deviceset="C" device="0603" package3d_urn="urn:adsk.eagle:package:19572011/3" override_package3d_urn="urn:adsk.eagle:package:19477979/2" override_package_urn="urn:adsk.eagle:footprint:23123/1" override_locally_modified="yes" value="10uF 10v"/>
 <part name="C3" library="_T_rcl" library_urn="urn:adsk.eagle:library:19571919" deviceset="C" device="0603" package3d_urn="urn:adsk.eagle:package:19572011/3" value="0.1uF 10V"/>
 <part name="C4" library="_T_rcl" library_urn="urn:adsk.eagle:library:19571919" deviceset="C" device="0603" package3d_urn="urn:adsk.eagle:package:19572011/3" value="10nF 16v"/>
@@
 <part name="U$1" library="_T_power" library_urn="urn:adsk.eagle:library:19572085" deviceset="+5V" device=""/>
 <part name="U$2" library="_T_power" library_urn="urn:adsk.eagle:library:19572085" deviceset="+5V" device=""/>
+<part name="C2" library="_T_rcl" library_urn="urn:adsk.eagle:library:19571919" deviceset="C" device="0603" package3d_urn="urn:adsk.eagle:package:19572011/3" value="10uF 10V"/>
 </parts>
 <sheets>
@@
 <attribute name="VALUE" x="254" y="182.88" size="1.778" layer="96" rot="R90"/>
 </instance>
-<instance part="C2" gate="G$1" x="256.54" y="175.26" smashed="yes" grouprefs="GYRO">
-<attribute name="NAME" x="258.953" y="175.514" size="1.778" layer="95" rot="R90"/>
-<attribute name="VALUE" x="253.619" y="171.704" size="1.778" layer="96" rot="R90"/>
-</instance>
 <instance part="C3" gate="G$1" x="248.92" y="175.26" smashed="yes" grouprefs="GYRO">
 <attribute name="NAME" x="251.333" y="175.514" size="1.778" layer="95" rot="R90"/>
@@
 <instance part="U$2" gate="G$1" x="142.24" y="66.04" smashed="yes">
 <attribute name="VALUE" x="139.7" y="60.96" size="1.778" layer="96" rot="R90"/>
+</instance>
+<instance part="C2" gate="G$1" x="256.54" y="175.26" smashed="yes">
+<attribute name="NAME" x="258.064" y="175.641" size="1.778" layer="95"/>
+<attribute name="VALUE" x="258.064" y="170.561" size="1.778" layer="96"/>
 </instance>
 </instances>
@@
 </segment>
 <segment>
-<pinref part="C2" gate="G$1" pin="2"/>
 <wire x1="254" y1="167.64" x2="256.54" y2="167.64" width="0.1524" layer="91" grouprefs="GYRO"/>
 <wire x1="256.54" y1="167.64" x2="256.54" y2="170.18" width="0.1524" layer="91" grouprefs="GYRO"/>
@@
 <junction x="254" y="167.64" grouprefs="GYRO"/>
 <pinref part="GND20" gate="G$1" pin="GND"/>
+<pinref part="C2" gate="G$1" pin="2"/>
 </segment>
 <segment>
@@
 <wire x1="248.92" y1="180.34" x2="256.54" y2="180.34" width="0.1524" layer="91" grouprefs="GYRO"/>
 <wire x1="256.54" y1="180.34" x2="256.54" y2="182.88" width="0.1524" layer="91" grouprefs="GYRO"/>
-<pinref part="C2" gate="G$1" pin="1"/>
 <wire x1="256.54" y1="177.8" x2="256.54" y2="180.34" width="0.1524" layer="91" grouprefs="GYRO"/>
 <junction x="256.54" y="180.34" grouprefs="GYRO"/>
@@
 <wire x1="228.6" y1="177.8" x2="228.6" y2="180.34" width="0.1524" layer="91" grouprefs="GYRO"/>
 <junction x="228.6" y="180.34" grouprefs="GYRO"/>
+<pinref part="C2" gate="G$1" pin="1"/>
 </segment>
 <segment>
@@
 will not be understood (or retained) with this version.
 </note>
-<note version="9.4" severity="warning">
-Since Version 9.4, EAGLE supports the overriding of 3D packages
-in schematics and board files. Those overridden 3d packages
-will not be understood (or retained) with this version.
-</note>
