File: hardware/ahrs/ahrs_v2.brd (EAGLE design)
At the start: 32 x 32 mm, 35 parts, among them J1 LINEAR_2_5040500291, J2 LINEAR_35040500391, J3 LINEAR_85040500891, U1 STM32G4_UFQFPN48_T1, U10 MCP2542FD, U11 LDFM33PUR, U2 LSM9DS1, X1 CRYSTAL_NX2016SA-24MHZ-EXS00A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

Commit message: Board rework
Parts:
- moved C12 30.8 mm to (18.1, 50.4)
- moved C13 30.8 mm to (21.9, 49.6)
- moved C14 30.8 mm to (19.4, 47.1)
- moved C15 30.8 mm to (31.5, 36.9)
- moved C16 30.8 mm to (37.2, 41.5)
- moved C37 30.8 mm to (20.7, 45.4)
- moved C38 30.8 mm to (43.5, 53.0)
- moved C39 30.8 mm to (39.7, 56.8)
- moved C40 30.8 mm to (42.3, 55.5)
- moved C42 30.8 mm to (34.6, 45.4)
- moved C1 30.8 mm to (15.6, 48.3)
- moved C11 22.8 mm to (7.83, 19.7), turned to 270 degrees
- moved R4 21.7 mm to (12.1, 8.56), turned to 180 degrees
- moved C41 18.8 mm to (7.62, 11.2)
- moved U11 16.5 mm to (24.9, 10.9)
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Routing:
- net GND: track 0.00 -> 4.64 mm, vias 0 -> 3
- net +3V3: track 0.00 -> 1.27 mm, vias 0 -> 1
- added copper zone on layer 2, net +3V3
- added copper zone on layer 15, net GND

Commit message: Restore after crash
Parts:
- added D1, D2, D3: (no value), _T_rcl:D0603
- added R1, R3: 22, _T_rcl:R0603
- added R2: 270, _T_rcl:R0603
- moved C40 53.6 mm to (1.80, 20.3)
- moved C38 52.6 mm to (4.40, 17.9), turned to 90 degrees
- moved C39 51.6 mm to (1.80, 21.8)
- moved C42 36.4 mm to (8.06, 20.6), turned to 270 degrees
- moved C12 32.7 mm to (27.6, 19.1)
- moved C1 31.6 mm to (27.8, 19.2)
- moved C13 30.7 mm to (27.3, 19.4)
- moved C15 29.3 mm to (9.01, 18.2)
- moved C14 29.1 mm to (27.5, 19.2)
- moved C37 24.8 mm to (10.4, 22.8)
- moved U11 24.0 mm to (1.89, 17.7)
- moved C16 23.3 mm to (27.7, 20.2)
- moved C36 13.4 mm to (1.50, 13.9)
- moved C4 10.9 mm to (4.40, 15.3), turned to 90 degrees
- moved C9 10.7 mm to (20.6, 9.23)
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Connections:
- new net LEDB: D1.2, U1.47
- new net LEDG: D3.2, U1.45
- new net LEDR: D2.2, U1.44
- new net LPUART1_RX: J3.P7
- new net LPUART1_TX: J3.P6
- new net LPUART_RX: U1.11
- new net LPUART_TX: U1.10
- new net N$6: D3.1, R3.2
- new net N$7: D2.1, R2.2
- new net N$8: D1.1, R1.2
- new net SPI3_CS: U1.12
- new net SPI3_MISO: U1.40
- new net SPI3_MOSI: U1.43
- new net SPI3_SCK: U1.39, U2.P$2
- new net SWCLK: J3.P3
- new net SWDIO: J3.P4, U1.36
- new net SWO: J3.P5, U1.41
- net +3V3: now also J3.P1
- net FDCAN1_RX: now also U1.33
- net FDCAN1_TX: now also U1.34
- net GND: now also J3.P8, R1.1, R2.1, R3.1
- net NRST: now also J3.P2
Routing:
- net +5V: track 0.00 -> 45.9 mm, vias 0 -> 2
- net GND: track 4.64 -> 44.0 mm, vias 3 -> 17
- net +3V3: track 1.27 -> 36.2 mm, vias 1 -> 10
- net FDCAN1_RX: track 0.00 -> 19.0 mm, vias 0 -> 2
- net FDCAN1_TX: track 0.00 -> 18.2 mm, vias 0 -> 2
- net NRST: track 0.00 -> 16.3 mm, vias 0 -> 2
- net N$11: track 0.00 -> 10.8 mm
- net N$12: track 0.00 -> 10.3 mm
- net N$1: track 0.00 -> 9.07 mm
- net N$3: track 0.00 -> 6.68 mm
- net N$2: track 0.00 -> 5.63 mm
- net N$16: track 0.00 -> 5.57 mm
- removed copper zone on layer 1, net +5V

Commit message: AHRS v2 layout complete
Parts:
- D1: value (none) -> 150060BS75000
- D2: value (none) -> 150060RS75000
- D3: value (none) -> 150060GS75000
- moved C1 4.63 mm to (30.4, 23.0), turned to 270 degrees
- moved C16 4.25 mm to (24.5, 23.1), turned to 270 degrees
- moved C12 4.08 mm to (26.5, 23.1), turned to 270 degrees
- moved C13 3.85 mm to (28.5, 23.1), turned to 270 degrees
- moved C14 3.02 mm to (24.5, 19.8), turned to 90 degrees
- moved U2 1.08 mm to (28.4, 18.8)
- moved C9 0.94 mm to (19.8, 8.73)
- moved C8 0.94 mm to (17.9, 8.74)
Connections:
- removed net LPUART_RX: U1.11
- removed net LPUART_TX: U1.10
- removed net MISO_AG: U2.P$5
- removed net MISO_M: U2.P$6
- removed net MOSI: U2.P$4
- removed net SPI3_CS: U1.12
- net CS_AG: now also U1.12
- net CS_M: now also U1.42
- net LEDB: now also U1.29; no longer U1.47
- net LEDG: now also U1.28; no longer U1.45
- net LEDR: now also U1.27; no longer U1.44
- net LPUART1_RX: now also U1.11
- net LPUART1_TX: now also U1.10
- net SPI3_MISO: now also U2.P$5, U2.P$6
- net SPI3_MOSI: now also U2.P$4
- net SWCLK: now also U1.37
Routing:
- net LPUART1_RX: track 0.00 -> 20.0 mm, vias 0 -> 2
- net CS_AG: track 0.00 -> 19.6 mm, vias 0 -> 2
- net SWDIO: track 0.00 -> 16.8 mm, vias 0 -> 2
- net SWCLK: track 0.00 -> 16.4 mm, vias 0 -> 2
- net LPUART1_TX: track 0.00 -> 16.2 mm, vias 0 -> 2
- net LEDR: track 0.00 -> 15.8 mm
- net GND: track 44.0 -> 58.9 mm, vias 17 -> 31
- net LEDG: track 0.00 -> 14.9 mm
- net LEDB: track 0.00 -> 14.6 mm
- net CS_M: track 0.00 -> 12.9 mm, vias 0 -> 2
- net +3V3: track 36.2 -> 48.7 mm, vias 10 -> 12
- net SPI3_MOSI: track 0.00 -> 11.1 mm, vias 0 -> 2
- net SWO: track 0.00 -> 10.8 mm
- net SPI3_SCK: track 0.00 -> 10.1 mm, vias 0 -> 2
- net SPI3_MISO: track 0.00 -> 9.15 mm
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
Commit message: Spacing
Parts:
- moved C42 0.51 mm to (7.56, 20.7)
- moved C37 0.50 mm to (10.4, 23.3)
- moved C15 0.20 mm to (9.01, 18.0)
Routing:
- net GND: track 58.9 -> 60.7 mm
- net N$2: track 5.63 -> 6.13 mm
- net SPI3_MISO: track 9.15 -> 9.34 mm, vias 0 -> 1

Commit message: Label movement
Parts:
- moved C39 1.80 mm to (1.80, 23.6)
- moved C40 1.80 mm to (1.80, 22.1)
Routing:
- net +3V3: track 48.7 -> 50.5 mm
