File: hardware/ahrs/ahrs_v2.sch (EAGLE design)
At the start: 34 parts, among them J2 LINEAR_35040500391, U1 STM32G4_UFQFPN48_T1, U10 MCP2542FD, U11 LDFM33PUR, U2 LSM9DS1, U9 STM32G4_UFQFPN48_T1, X1 CRYSTAL_NX2016SA-24MHZ-EXS00A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

Commit message: AHRS V2 work
Parts:
- removed U9: STM32G4_UFQFPN48_T1, _T_ic:STM32G4_UFQFPN48_T1
- added J1: LINEAR_2_5040500291, _T_conn:LINEAR_2_5040500291
- added J3: LINEAR_85040500891, _T_conn:LINEAR_85040500891
Connections:
- net +3V3: now also U1B.VBAT, U1B.VDD, U1B.VDD_2, U1B.VDD_3; no longer U9B.VBAT, U9B.VDD, U9B.VDD_2, U9B.VDD_3
- net +5V: now also J1.P1
- net GND: now also J1.P2, U1B.EPAD; no longer U9B.EPAD
- net N$1: now also U1B.VREF+; no longer U9B.VREF+
- net N$16: now also U1B.VDDA; no longer U9B.VDDA
Other:
- moved on the sheet: C1, C12, C13, C14, C16, U2

Commit message: Restore after crash
Parts:
- added D1, D2, D3: (no value), _T_rcl:LED_0603
- added R1, R3: 22, _T_rcl:R0603
- added R2: 270, _T_rcl:R0603
Connections:
- new net LEDB: D1.A, U1A.PB9
- new net LEDG: D3.A, U1A.PB7
- new net LEDR: D2.A, U1A.PB6
- new net LPUART1_RX: J3.P7
- new net LPUART1_TX: J3.P6
- new net LPUART_RX: U1A.PA3
- new net LPUART_TX: U1A.PA2
- new net N$6: D3.C, R3.2
- new net N$7: D2.C, R2.2
- new net N$8: D1.C, R1.2
- new net SPI3_CS: U1A.PA4
- new net SPI3_MISO: U1A.PC11
- new net SPI3_MOSI: U1A.PB5
- new net SPI3_SCK: U1A.PC10, U2.SCL/SPC
- new net SWCLK: J3.P3
- new net SWDIO: J3.P4, U1A.PA13
- new net SWO: J3.P5, U1A.PB3
- net +3V3: now also J3.P1
- net FDCAN1_RX: now also U1A.PA11
- net FDCAN1_TX: now also U1A.PA12
- net GND: now also J3.P8, R1.1, R2.1, R3.1
- net NRST: now also J3.P2
Other:
- moved on the sheet: J3

Commit message: AHRS v2 layout complete
Parts:
- D1: value (none) -> 150060BS75000
- D2: value (none) -> 150060RS75000
- D3: value (none) -> 150060GS75000
Connections:
- removed net LPUART_RX: U1A.PA3
- removed net LPUART_TX: U1A.PA2
- removed net MISO_AG: U2.SDO_A/G
- removed net MISO_M: U2.SDO_M
- removed net MOSI: U2.SDA/SDI/SDO
- removed net SPI3_CS: U1A.PA4
- net CS_AG: now also U1A.PA4
- net CS_M: now also U1A.PB4
- net LEDB: now also U1A.PC6; no longer U1A.PB9
- net LEDG: now also U1A.PB15; no longer U1A.PB7
- net LEDR: now also U1A.PB14; no longer U1A.PB6
- net LPUART1_RX: now also U1A.PA3
- net LPUART1_TX: now also U1A.PA2
- net SPI3_MISO: now also U2.SDO_A/G, U2.SDO_M
- net SPI3_MOSI: now also U2.SDA/SDI/SDO
- net SWCLK: now also U1A.PA14
