File: hardware/BLDC/bldc.sch (EAGLE design)
At the start: 84 parts, among them J1 PWR_2_XT30PW-M, J2 LINEAR_3_JST_PH_RA, J3 LINEAR_8_JST_PH_RA, U1 MA702, U10 MCP2542FD, U11 LDFM33PUR, U2 DRV8323RS, U3 TPN7R006PL, U4 TPN7R006PL, U5 TPN7R006PL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

Commit message: BoM consolidation and package standardization
Parts:
- C13, C34, C35: device _T_rcl:C0603 -> _T_rcl:C0402
- C14: value 2.2uF 10V -> 2.2uF 50V
- C36, C41: value 0.1uF 10V -> 100nF 10V
Changed lines of the file:
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@@
 <part name="GND9" library="_T_power" library_urn="urn:adsk.eagle:library:19572085" deviceset="GND" device=""/>
 <part name="GND10" library="_T_power" library_urn="urn:adsk.eagle:library:19572085" deviceset="GND" device=""/>
-<part name="C13" library="_T_rcl" library_urn="urn:adsk.eagle:library:19571919" deviceset="C" device="0603" package3d_urn="urn:adsk.eagle:package:19572011/3" value="100nF 10V"/>
+<part name="C13" library="_T_rcl" library_urn="urn:adsk.eagle:library:19571919" deviceset="C" device="0402" package3d_urn="urn:adsk.eagle:package:19572013/4" value="100nF 10V"/>
 <part name="L2" library="_T_rcl" library_urn="urn:adsk.eagle:library:19571919" deviceset="L" device="_SDR0302" package3d_urn="urn:adsk.eagle:package:20294118/5" value="22uH Bourns"/>
 <part name="R2" library="_T_rcl" library_urn="urn:adsk.eagle:library:19571919" deviceset="R" device="0402" package3d_urn="urn:adsk.eagle:package:19572014/3" value="100k"/>
 <part name="R3" library="_T_rcl" library_urn="urn:adsk.eagle:library:19571919" deviceset="R" device="0402" package3d_urn="urn:adsk.eagle:package:19572014/3" value="100k"/>
 <part name="GND11" library="_T_power" library_urn="urn:adsk.eagle:library:19572085" deviceset="GND" device=""/>
-<part name="C14" library="_T_rcl" library_urn="urn:adsk.eagle:library:19571919" deviceset="C" device="0603" package3d_urn="urn:adsk.eagle:package:19572011/3" value="2.2uF 10V"/>
+<part name="C14" library="_T_rcl" library_urn="urn:adsk.eagle:library:19571919" deviceset="C" device="0603" package3d_urn="urn:adsk.eagle:package:19572011/3" value="2.2uF 50V"/>
 <part name="GND12" library="_T_power" library_urn="urn:adsk.eagle:library:19572085" deviceset="GND" device=""/>
 <part name="D1" library="_T_rcl" library_urn="urn:adsk.eagle:library:19571919" deviceset="SCHOTTKY" device="_SOD123" package3d_urn="urn:adsk.eagle:package:20295471/2"/>
@@
 <part name="GND17" library="_T_power" library_urn="urn:adsk.eagle:library:19572085" deviceset="GND" device=""/>
 <part name="C33" library="_T_rcl" library_urn="urn:adsk.eagle:library:19571919" deviceset="C" device="0402" package3d_urn="urn:adsk.eagle:package:19572013/4" value="47nF 50v"/>
-<part name="C34" library="_T_rcl" library_urn="urn:adsk.eagle:library:19571919" deviceset="C" device="0603" package3d_urn="urn:adsk.eagle:package:19572011/3" value="1uf 10v"/>
+<part name="C34" library="_T_rcl" library_urn="urn:adsk.eagle:library:19571919" deviceset="C" device="0402" package3d_urn="urn:adsk.eagle:package:19572013/4" value="1uf 10v"/>
 <part name="GND18" library="_T_power" library_urn="urn:adsk.eagle:library:19572085" deviceset="GND" device=""/>
-<part name="C35" library="_T_rcl" library_urn="urn:adsk.eagle:library:19571919" deviceset="C" device="0603" package3d_urn="urn:adsk.eagle:package:19572011/3" value="1uf 10v"/>
-<part name="R5" library="_T_rcl" library_urn="urn:adsk.eagle:library:19571919" deviceset="R_SENSE" device="_1210" package3d_urn="urn:adsk.eagle:package:16502583/3" value="0.001"/>
-<part name="R6" library="_T_rcl" library_urn="urn:adsk.eagle:library:19571919" deviceset="R_SENSE" device="_1210" package3d_urn="urn:adsk.eagle:package:16502583/3" value="0.001"/>
-<part name="R7" library="_T_rcl" library_urn="urn:adsk.eagle:library:19571919" deviceset="R_SENSE" device="_1210" package3d_urn="urn:adsk.eagle:package:16502583/3" value="0.001"/>
+<part name="C35" library="_T_rcl" library_urn="urn:adsk.eagle:library:19571919" deviceset="C" device="0402" package3d_urn="urn:adsk.eagle:package:19572013/4" value="1uf 10v"/>
+<part name="R5" library="_T_rcl" library_urn="urn:adsk.eagle:library:19571919" deviceset="R_SENSE" device="_1210" package3d_urn="urn:adsk.eagle:package:16502583/4" value="0.001"/>
+<part name="R6" library="_T_rcl" library_urn="urn:adsk.eagle:library:19571919" deviceset="R_SENSE" device="_1210" package3d_urn="urn:adsk.eagle:package:16502583/4" value="0.001"/>
+<part name="R7" library="_T_rcl" library_urn="urn:adsk.eagle:library:19571919" deviceset="R_SENSE" device="_1210" package3d_urn="urn:adsk.eagle:package:16502583/4" value="0.001"/>
 <part name="GND19" library="_T_power" library_urn="urn:adsk.eagle:library:19572085" deviceset="GND" device=""/>
 <part name="GND20" library="_T_power" library_urn="urn:adsk.eagle:library:19572085" deviceset="GND" device=""/>
@@
 <part name="GND23" library="_T_power" library_urn="urn:adsk.eagle:library:19572085" deviceset="GND" device=""/>
 <part name="+3V11" library="_T_power" library_urn="urn:adsk.eagle:library:19572085" deviceset="+3V3" device=""/>
-<part name="C36" library="_T_rcl" library_urn="urn:adsk.eagle:library:19571919" deviceset="C" device="0402" package3d_urn="urn:adsk.eagle:package:19572013/4" value="0.1uF 10V"/>
+<part name="C36" library="_T_rcl" library_urn="urn:adsk.eagle:library:19571919" deviceset="C" device="0402" package3d_urn="urn:adsk.eagle:package:19572013/4" value="100nF 10V"/>
 <part name="+5V3" library="_T_power" library_urn="urn:adsk.eagle:library:19572085" deviceset="+5V" device=""/>
 <part name="GND24" library="_T_power" library_urn="urn:adsk.eagle:library:19572085" deviceset="GND" device=""/>
-<part name="C41" library="_T_rcl" library_urn="urn:adsk.eagle:library:19571919" deviceset="C" device="0402" package3d_urn="urn:adsk.eagle:package:19572013/4" value="0.1uF 10V"/>
+<part name="C41" library="_T_rcl" library_urn="urn:adsk.eagle:library:19571919" deviceset="C" device="0402" package3d_urn="urn:adsk.eagle:package:19572013/4" value="100nF 10V"/>
 <part name="+3V12" library="_T_power" library_urn="urn:adsk.eagle:library:19572085" deviceset="+3V3" device=""/>
 <part name="C42" library="_T_rcl" library_urn="urn:adsk.eagle:library:19571919" deviceset="C" device="0402" package3d_urn="urn:adsk.eagle:package:19572013/4" value="6.8pF 10V"/>

Commit message: Oops, no longer grounded INLx
Parts:
- C14: value 2.2uF 50V -> 10uF 50V
- R12: value 5 -> 22
Connections:
- net DRV_ENABLE: now also U2.INLA, U2.INLB, U2.INLC
- net GND: no longer U2.INLA, U2.INLB, U2.INLC
Other:
- moved on the sheet: C1, C10, C11, C16, C17, C18, C19, C2, C20, C21, C22, C23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

Commit message: Fixes prior to reworking SPI2>SPI3
Parts:
- R13: value 65 -> 270
- R14: value 5 -> 22
- R2: value 100k -> 54.9k 1%
- R3: value 100k -> 10k 1%
Connections:
- net VBUS_SENSE renamed VBAT_SENSE
- removed net CAL: U2.CAL
- net GND: now also U9A.PB8-BOOT0
Other:
- moved on the sheet: C35
Changed lines of the file:
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@@
 <part name="C13" library="_T_rcl" library_urn="urn:adsk.eagle:library:19571919" deviceset="C" device="0402" package3d_urn="urn:adsk.eagle:package:19572013/4" value="100nF 10V"/>
 <part name="L2" library="_T_rcl" library_urn="urn:adsk.eagle:library:19571919" deviceset="L" device="_SDR0302" package3d_urn="urn:adsk.eagle:package:20294118/5" value="22uH Bourns"/>
-<part name="R2" library="_T_rcl" library_urn="urn:adsk.eagle:library:19571919" deviceset="R" device="0402" package3d_urn="urn:adsk.eagle:package:19572014/3" value="100k"/>
-<part name="R3" library="_T_rcl" library_urn="urn:adsk.eagle:library:19571919" deviceset="R" device="0402" package3d_urn="urn:adsk.eagle:package:19572014/3" value="100k"/>
+<part name="R2" library="_T_rcl" library_urn="urn:adsk.eagle:library:19571919" deviceset="R" device="0402" package3d_urn="urn:adsk.eagle:package:19572014/3" value="54.9k 1%"/>
+<part name="R3" library="_T_rcl" library_urn="urn:adsk.eagle:library:19571919" deviceset="R" device="0402" package3d_urn="urn:adsk.eagle:package:19572014/3" value="10k 1%"/>
 <part name="GND11" library="_T_power" library_urn="urn:adsk.eagle:library:19572085" deviceset="GND" device=""/>
 <part name="C14" library="_T_rcl" library_urn="urn:adsk.eagle:library:19571919" deviceset="C" device="0603" package3d_urn="urn:adsk.eagle:package:19572011/3" value="10uF 50V"/>
@@
 <part name="D4" library="_T_rcl" library_urn="urn:adsk.eagle:library:19571919" deviceset="LED" device="_0603" package3d_urn="urn:adsk.eagle:package:19545722/3" value="150060BS75000"/>
 <part name="R12" library="_T_rcl" library_urn="urn:adsk.eagle:library:19571919" deviceset="R" device="0402" package3d_urn="urn:adsk.eagle:package:19572014/3" value="22"/>
-<part name="R13" library="_T_rcl" library_urn="urn:adsk.eagle:library:19571919" deviceset="R" device="0402" package3d_urn="urn:adsk.eagle:package:19572014/3" value="65"/>
-<part name="R14" library="_T_rcl" library_urn="urn:adsk.eagle:library:19571919" deviceset="R" device="0402" package3d_urn="urn:adsk.eagle:package:19572014/3" value="5"/>
+<part name="R13" library="_T_rcl" library_urn="urn:adsk.eagle:library:19571919" deviceset="R" device="0402" package3d_urn="urn:adsk.eagle:package:19572014/3" value="270"/>
+<part name="R14" library="_T_rcl" library_urn="urn:adsk.eagle:library:19571919" deviceset="R" device="0402" package3d_urn="urn:adsk.eagle:package:19572014/3" value="22"/>
 <part name="GND28" library="_T_power" library_urn="urn:adsk.eagle:library:19572085" deviceset="GND" device=""/>
+<part name="GND3" library="_T_power" library_urn="urn:adsk.eagle:library:19572085" deviceset="GND" device=""/>
+<part name="GND29" library="_T_power" library_urn="urn:adsk.eagle:library:19572085" deviceset="GND" device=""/>
 </parts>
 <sheets>
@@
 <attribute name="VALUE" x="92.964" y="117.221" size="1.778" layer="96"/>
 </instance>
-<instance part="GND18" gate="G$1" x="78.74" y="132.08" smashed="yes" grouprefs="GATE_DRIVER_DRV8323RS">
-<attribute name="VALUE" x="76.835" y="128.905" size="1.778" layer="96"/>
-</instance>
-<instance part="C35" gate="G$1" x="78.74" y="142.24" smashed="yes" grouprefs="GATE_DRIVER_DRV8323RS">
-<attribute name="NAME" x="80.264" y="142.621" size="1.778" layer="95"/>
-<attribute name="VALUE" x="80.264" y="137.541" size="1.778" layer="96"/>
+<instance part="GND18" gate="G$1" x="99.06" y="127" smashed="yes" grouprefs="GATE_DRIVER_DRV8323RS">
+<attribute name="VALUE" x="97.155" y="123.825" size="1.778" layer="96"/>
+</instance>
+<instance part="C35" gate="G$1" x="76.2" y="76.2" smashed="yes" grouprefs="GATE_DRIVER_DRV8323RS">
+<attribute name="NAME" x="77.724" y="76.581" size="1.778" layer="95"/>
+<attribute name="VALUE" x="77.724" y="71.501" size="1.778" layer="96"/>
 </instance>
 <instance part="R5" gate="G$1" x="223.52" y="76.2" smashed="yes" rot="R270" grouprefs="H_BRIDGE">
@@
 <instance part="GND28" gate="G$1" x="27.94" y="147.32" smashed="yes" grouprefs="LED_INFO">
 <attribute name="VALUE" x="26.035" y="149.225" size="1.778" layer="96"/>
+</instance>
+<instance part="GND3" gate="G$1" x="76.2" y="66.04" smashed="yes" grouprefs="GATE_DRIVER_DRV8323RS">
+<attribute name="VALUE" x="74.295" y="62.865" size="1.778" layer="96"/>
+</instance>
+<instance part="GND29" gate="G$1" x="-73.66" y="58.42" smashed="yes" grouprefs="UC_STM32G4">
+<attribute name="VALUE" x="-75.565" y="55.245" size="1.778" layer="96"/>
 </instance>
 </instances>
@@
 </segment>
 <segment>
-<pinref part="C35" gate="G$1" pin="1"/>
-<wire x1="78.74" y1="144.78" x2="78.74" y2="147.32" width="0.1524" layer="91" grouprefs="GATE_DRIVER_DRV8323RS"/>
-<label x="78.74" y="147.32" size="1.27" layer="95" rot="R180" xref="yes" grouprefs="GATE_DRIVER_DRV8323RS"/>
-</segment>
-<segment>
 <pinref part="R8" gate="G$1" pin="2"/>
 <wire x1="157.48" y1="119.38" x2="157.48" y2="121.92" width="0.1524" layer="91" grouprefs="GATE_DRIVER_DRV8323RS"/>
@@
 <segment>
 <pinref part="U2" gate="G$1" pin="VREF"/>
-<wire x1="101.6" y1="78.74" x2="99.06" y2="78.74" width="0.1524" layer="91" grouprefs="GATE_DRIVER_DRV8323RS"/>
-<label x="99.06" y="78.74" size="1.27" layer="95" rot="R180" xref="yes" grouprefs="GATE_DRIVER_DRV8323RS"/>
+<wire x1="101.6" y1="78.74" x2="76.2" y2="78.74" width="0.1524" layer="91" grouprefs="GATE_DRIVER_DRV8323RS"/>
+<label x="73.66" y="78.74" size="1.27" layer="95" rot="R180" xref="yes" grouprefs="GATE_DRIVER_DRV8323RS"/>
+<pinref part="C35" gate="G$1" pin="1"/>
+<wire x1="76.2" y1="78.74" x2="73.66" y2="78.74" width="0.1524" layer="91" grouprefs="GATE_DRIVER_DRV8323RS"/>
+<junction x="76.2" y="78.74" grouprefs="GATE_DRIVER_DRV8323RS"/>
 </segment>
 <segment>
@@
 </segment>
 <segment>
-<pinref part="GND18" gate="G$1" pin="GND"/>
-<wire x1="78.74" y1="134.62" x2="78.74" y2="137.16" width="0.1524" layer="91" grouprefs="GATE_DRIVER_DRV8323RS"/>
-<pinref part="C35" gate="G$1" pin="2"/>
-<pinref part="U2" gate="G$1" pin="DGND"/>
-<wire x1="101.6" y1="129.54" x2="86.36" y2="129.54" width="0.1524" layer="91" grouprefs="GATE_DRIVER_DRV8323RS"/>
-<wire x1="86.36" y1="129.54" x2="86.36" y2="137.16" width="0.1524" layer="91" grouprefs="GATE_DRIVER_DRV8323RS"/>
-<wire x1="86.36" y1="137.16" x2="78.74" y2="137.16" width="0.1524" layer="91" grouprefs="GATE_DRIVER_DRV8323RS"/>
-<junction x="78.74" y="137.16" grouprefs="GATE_DRIVER_DRV8323RS"/>
-</segment>
-<segment>
 <pinref part="R7" gate="G$1" pin="2"/>
 <pinref part="GND21" gate="G$1" pin="GND"/>
@@
 <pinref part="R13" gate="G$1" pin="1"/>
 <wire x1="27.94" y1="152.4" x2="27.94" y2="149.86" width="0.1524" layer="91" grouprefs="LED_INFO"/>
+</segment>
+<segment>
+<pinref part="U2" gate="G$1" pin="DGND"/>
+<pinref part="GND18" gate="G$1" pin="GND"/>
+<wire x1="101.6" y1="129.54" x2="99.06" y2="129.54" width="0.1524" layer="91" grouprefs="GATE_DRIVER_DRV8323RS"/>
+</segment>
+<segment>
+<pinref part="GND3" gate="G$1" pin="GND"/>
+<pinref part="C35" gate="G$1" pin="2"/>
+<wire x1="76.2" y1="68.58" x2="76.2" y2="71.12" width="0.1524" layer="91" grouprefs="GATE_DRIVER_DRV8323RS"/>
+</segment>
+<segment>
+<pinref part="U9" gate="A" pin="PB8-BOOT0"/>
+<pinref part="GND29" gate="G$1" pin="GND"/>
+<wire x1="-58.42" y1="60.96" x2="-73.66" y2="60.96" width="0.1524" layer="91" grouprefs="UC_STM32G4"/>
 </segment>
 </net>
@@
 <pinref part="U2" gate="G$1" pin="DVDD"/>
 <wire x1="101.6" y1="124.46" x2="91.44" y2="124.46" width="0.1524" layer="91" grouprefs="GATE_DRIVER_DRV8323RS"/>
-<wire x1="91.44" y1="124.46" x2="81.28" y2="124.46" width="0.1524" layer="91" grouprefs="GATE_DRIVER_DRV8323RS"/>
 <pinref part="C34" gate="G$1" pin="1"/>
-<junction x="91.44" y="124.46" grouprefs="GATE_DRIVER_DRV8323RS"/>
-<label x="81.28" y="124.46" size="1.27" layer="95" rot="R180" xref="yes" grouprefs="GATE_DRIVER_DRV8323RS"/>
 </segment>
 </net>
@@
 <wire x1="101.6" y1="101.6" x2="99.06" y2="101.6" width="0.1524" layer="91" grouprefs="GATE_DRIVER_DRV8323RS"/>
 <junction x="99.06" y="101.6" grouprefs="GATE_DRIVER_DRV8323RS"/>
-<label x="96.52" y="96.52" size="1.27" layer="95" rot="R180" xref="yes"/>
+<label x="96.52" y="96.52" size="1.27" layer="95" rot="R180" xref="yes" grouprefs="GATE_DRIVER_DRV8323RS"/>
 </segment>
 </net>
@@
 </segment>
 </net>
-<net name="CAL" class="0">
-<segment>
-<pinref part="U2" gate="G$1" pin="CAL"/>
-<wire x1="101.6" y1="66.04" x2="99.06" y2="66.04" width="0.1524" layer="91" grouprefs="GATE_DRIVER_DRV8323RS"/>
-<label x="99.06" y="66.04" size="1.27" layer="95" rot="R180" xref="yes" grouprefs="GATE_DRIVER_DRV8323RS"/>
-</segment>
-</net>
 <net name="SENSE_A" class="0">
 <segment>
@@
 </segment>
 </net>
-<net name="VBUS_SENSE" class="0">
+<net name="VBAT_SENSE" class="0">
 <segment>
 <pinref part="U9" gate="A" pin="PB12"/>
