File: bldc/hardware/v2.0/bldc_octo.brd (EAGLE design)
At the start: 60 x 60 mm, 11 parts, among them J1 PWR_2_XT30PW-M, J2 LINEAR_3_MOLEX_5023520300, J3 LINEAR_3_AMASS_MR30PW-M, U1 MA702, U2 STM32H723VGT6, U3 DRV8323RS, U4 MCP2542FD, X1 CRYSTAL_NX2016SA-24MHZ-EXS00A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

Commit message: Going to start can
Parts:
- added Q1, Q2, Q3: CSD88599Q5DC, _T_transistors:CSD88599Q5DC
- J2: value LINEAR_3_MOLEX_5023520300 -> LINEAR_3_MOLEX_5055670381; device _T_conn:MOLEX_5023520300 -> _T_conn:MOLEX_5055670381
- moved J2 0.32 mm to (35.9, 0.00), turned to 180 degrees
Connections:
- new net N$5: Q1.VIN$1, Q1.VIN$10, Q1.VIN$11, Q1.VIN$2, Q1.VIN$3, Q1.VIN$4, Q1.VIN$5, Q1.VIN$6, Q1.VIN$7, Q1.VIN$8, Q1.VIN$9, Q2.VIN$1, Q2.VIN$10, Q2.VIN$11, Q2.VIN$2, Q2.VIN$3, Q2.VIN$4, Q2.VIN$5, Q2.VIN$6, Q2.VIN$7, Q2.VIN$8, Q2.VIN$9, Q3.VIN$1, Q3.VIN$10, Q3.VIN$11, Q3.VIN$2, Q3.VIN$3, Q3.VIN$4, Q3.VIN$5, Q3.VIN$6, Q3.VIN$7, Q3.VIN$8, Q3.VIN$9
- net GND: now also J2.PIN3; no longer J2.P$3
- net N$1: now also J2.PIN1; no longer J2.P$1
- net N$2: now also J2.PIN2; no longer J2.P$2
